File: mcu/KiCad/Ethernet_PHY.sch (KiCad schematic (older format))
At the start: 44 parts, among them IC16 TPD4E001DRLR, IC17 DP83848CVV_NOPB, X6 LMJTAB881243M-L

Commit message: Kicad-ised schematic, fixed import errors
Basic stuff like pin functions not assigned, and moving to heirarchial labels instead of global,
Connections:
- wire segments 228 -> 229
- no-connect marks 0 -> 7
Changed lines of the file:
@@
 $Descr User 12095 8535
 encoding utf-8
-Sheet 6 6
+Sheet 4 6
 Title "EEZ DIB MUC"
 Date ""
@@
 	7400 1500 7400 1600
 Connection ~ 7400 1500
-Text GLabel 7600 1500 0    10   BiDi ~ 0
-GND
 Wire Wire Line
 	7300 2400 7200 2400
 Wire Wire Line
 	7200 2500 7200 2400
-Text GLabel 7300 2400 0    10   BiDi ~ 0
-GND
 Wire Wire Line
 	8100 2500 8000 2500
 Wire Wire Line
 	8000 2600 8000 2500
-Text GLabel 8100 2500 0    10   BiDi ~ 0
-GND
 Wire Wire Line
 	8100 3300 8000 3300
 Wire Wire Line
 	8000 3400 8000 3300
-Text GLabel 8100 3300 0    10   BiDi ~ 0
-GND
 Wire Wire Line
 	7500 3300 7600 3300
 Wire Wire Line
 	7600 3400 7600 3300
-Text GLabel 7500 3300 0    10   BiDi ~ 0
-GND
 Wire Wire Line
 	9400 3900 9000 3900
 Wire Wire Line
 	9000 3900 9000 4000
-Text GLabel 9400 3900 0    10   BiDi ~ 0
-GND
 Wire Wire Line
 	5800 4900 5800 5000
@@
 Connection ~ 6200 5000
 Connection ~ 6000 5000
-Text GLabel 5800 4900 0    10   BiDi ~ 0
-GND
 Wire Wire Line
 	5000 5100 5200 5100
@@
 Connection ~ 5200 5400
 Connection ~ 5200 5500
-Text GLabel 5000 5100 0    10   BiDi ~ 0
-GND
 Wire Wire Line
 	2900 6000 2500 6000
@@
 Connection ~ 2500 6000
 Connection ~ 2900 6000
-Text GLabel 2900 6000 0    10   BiDi ~ 0
-GND
 Wire Wire Line
 	1300 3300 1300 3200
@@
 	1400 3200 1300 3200
 Connection ~ 1300 3200
-Text GLabel 1300 3300 0    10   BiDi ~ 0
-GND
 Wire Wire Line
 	3200 5600 2900 5600
@@
 	2900 5600 2900 5300
 Connection ~ 2900 5600
-Text GLabel 3200 5600 0    10   BiDi ~ 0
-+3V3
 Wire Wire Line
 	3200 5500 2500 5500
@@
 	2500 5500 2500 5300
 Connection ~ 2500 5500
-Text GLabel 3200 5500 0    10   BiDi ~ 0
-+3V3
 Wire Wire Line
 	1500 5400 1400 5400
 Wire Wire Line
 	1400 5400 1400 5300
-Text GLabel 1500 5400 0    10   BiDi ~ 0
-+3V3
 Wire Wire Line
 	6700 3100 6800 3100
@@
 Connection ~ 6800 3300
 Connection ~ 6800 3100
-Text GLabel 6700 3100 0    10   BiDi ~ 0
-+3V3
 Wire Wire Line
 	9400 4300 9100 4300
@@
 	9100 4600 9100 4300
 Connection ~ 9100 4300
-Text GLabel 9400 4300 0    10   BiDi ~ 0
-+3V3
 Wire Wire Line
 	2600 3500 2500 3500
@@
 	5500 5100 5500 5000
 Connection ~ 5500 5000
-Text GLabel 5400 5000 0    10   BiDi ~ 0
-+3V3
 Wire Wire Line
 	3100 1600 3100 1700
@@
 	7400 1200 7400 1100
 Connection ~ 7400 1200
-Text GLabel 7600 1200 0    10   BiDi ~ 0
-+3V3
-Wire Wire Line
-	1200 2600 2000 2600
-Text GLabel 1200 2600 2    50   BiDi ~ 0
-ETH_TX_EN
-Wire Wire Line
-	1200 2700 2000 2700
-Text GLabel 1200 2700 2    50   BiDi ~ 0
-ETH_RX_CLK
-Wire Wire Line
-	1200 2800 2000 2800
-Text GLabel 1200 2800 2    50   BiDi ~ 0
-ETH_RX_DV
-Wire Wire Line
-	2200 4100 1200 4100
-Text GLabel 1200 4100 2    50   BiDi ~ 0
-ETH_RXD0
-Wire Wire Line
-	1200 4200 2200 4200
-Text GLabel 1200 4200 2    50   BiDi ~ 0
-ETH_RXD1
-Wire Wire Line
-	1200 4300 2200 4300
-Text GLabel 1200 4300 2    50   BiDi ~ 0
-ETH_RXD2
-Wire Wire Line
-	1200 4400 2200 4400
-Text GLabel 1200 4400 2    50   BiDi ~ 0
-ETH_RXD3
-Wire Wire Line
-	1200 4600 2200 4600
-Text GLabel 1200 4600 2    50   BiDi ~ 0
-ETH_TXD0
-Wire Wire Line
-	1200 4700 2200 4700
-Text GLabel 1200 4700 2    50   BiDi ~ 0
-ETH_TXD1
-Wire Wire Line
-	1200 4800 2200 4800
-Text GLabel 1200 4800 2    50   BiDi ~ 0
-ETH_TXD2
-Wire Wire Line
-	1200 4900 2200 4900
-Text GLabel 1200 4900 2    50   BiDi ~ 0
-ETH_TXD3
-Wire Wire Line
-	1200 3800 3200 3800
-Text GLabel 1200 3800 2    50   BiDi ~ 0
-~RESET
+Wire Wire Line
+	1700 2600 2000 2600
+Wire Wire Line
+	1700 2700 2000 2700
+Wire Wire Line
+	1700 2800 2000 2800
+Wire Wire Line
+	2200 4100 1650 4100
+Wire Wire Line
+	1650 4200 2200 4200
+Wire Wire Line
+	1650 4300 2200 4300
+Wire Wire Line
+	1650 4400 2200 4400
+Wire Wire Line
+	1650 4600 2200 4600
+Wire Wire Line
+	1650 4700 2200 4700
+Wire Wire Line
+	1650 4800 2200 4800
+Wire Wire Line
+	1650 4900 2200 4900
+Wire Wire Line
+	1650 3800 3200 3800
 Wire Wire Line
 	2000 3400 2000 3700
@@
 Connection ~ 2000 3700
 Wire Wire Line
-	1200 2300 3000 2300
+	1700 2300 3000 2300
 Wire Wire Line
 	3000 2300 3000 2500
 Wire Wire Line
 	3000 2500 3200 2500
-Text GLabel 1200 2300 2    50   BiDi ~ 0
-ETH_MDC
-Wire Wire Line
-	1200 2200 3100 2200
+Wire Wire Line
+	1700 2200 3100 2200
 Wire Wire Line
 	3100 2200 3100 2400
@@
 Wire Wire Line
 	3100 2200 3100 2100
-Text GLabel 1200 2200 2    50   BiDi ~ 0
-ETH_MDIO
 Connection ~ 3100 2200
 Wire Wire Line
-	1200 2500 2000 2500
-Text GLabel 1200 2500 2    50   BiDi ~ 0
-ETH_TX_CLK
+	1700 2500 2000 2500
 Wire Wire Line
 	5000 4300 5400 4300
@@
 Connection ~ 6600 4300
 Wire Wire Line
-	3200 5400 2100 5400
+	3200 5400 2300 5400
 Wire Wire Line
 	2100 5400 2100 5600
@@
 	8400 2500 8400 2400
 Connection ~ 8400 2500
-Text Label 8400 2500 0    10   ~ 0
-+3V3(A)
 Wire Wire Line
 	8400 3300 9400 3300
@@
 	8400 3300 8400 3200
 Connection ~ 8400 3300
-Text Label 8400 3300 0    10   ~ 0
-+3V3(A)
 Wire Wire Line
 	7100 3300 7200 3300
@@
 	9400 4800 7700 4800
 Wire Wire Line
-	1200 2000 2000 2000
-Text GLabel 1200 2000 2    50   BiDi ~ 0
-MCLK_25
+	1700 2000 2000 2000
 Wire Wire Line
 	3200 2600 2900 2600
@@
 	2900 2000 2900 2600
 Wire Wire Line
-	1200 3900 1900 3900
+	1650 3900 1900 3900
 Wire Wire Line
 	1900 3400 1900 3900
 Wire Wire Line
 	2200 3900 1900 3900
-Text GLabel 1200 3900 2    50   BiDi ~ 0
-ETH_CRS
 Connection ~ 1900 3900
 Wire Wire Line
@@
 Wire Wire Line
 	9400 4000 9200 4000
-Text GLabel 9400 4000 0    10   BiDi ~ 0
-PE
 Wire Wire Line
 	3000 3200 3200 3200
@@
 	3200 3600 2600 3600
 Wire Wire Line
-	2200 3600 1200 3600
-Text GLabel 1200 3600 2    50   BiDi ~ 0
-ETH_COL
+	2200 3600 1650 3600
 Wire Wire Line
 	2600 4400 3200 4400
@@
 	2600 3900 3200 3900
 Wire Wire Line
-	1700 3700 1200 3700
-Text GLabel 1200 3700 2    50   BiDi ~ 0
-SPI5_IRQ
+	1700 3700 1650 3700
 $Comp
 L EEZ_DIB_MCU_r1B1-eagle-import:DINA4_L #FRAME5
@@
 $EndComp
 $Comp
-L EEZ_DIB_MCU_r1B1-eagle-import:C-EUC0603 C64
-U 1 0 B6C25B1D
-P 5800 4700
-AR Path="/B6C25B1D" Ref="C64"  Part="1"
-AR Path="/5B8E25B8/B6C25B1D" Ref="C64"  Part="1"
-F 0 "C64" H 5715 4735 59  0000 R TNN
-F 1 "100n" H 5715 4660 59  0000 R TNN
-F 2 "EEZ DIB MCU r1B1:C0603" H 5800 4700 50  0001 C CNN
-F 3 "" H 5800 4700 50  0001 C CNN
-	1    5800 4700
-	-1   0    0    -1
-$EndComp
-$Comp
 L EEZ_DIB_MCU_r1B1-eagle-import:C-EUC0603 C65
 U 1 0 E7D5C9F7
@@
 AR Path="/5B8E25B8/F72700C4" Ref="#+3V022"  Part="1"
 F 0 "#+3V022" H 2900 5200 50  0001 C CNN
-F 1 "+3V3" V 2775 5225 59  0000 L BNN
+F 1 "+3V3" H 2750 5200 59  0000 L BNN
 F 2 "" H 2900 5200 50  0001 C CNN
 F 3 "" H 2900 5200 50  0001 C CNN
@@
 AR Path="/5B8E25B8/7D977A11" Ref="#+3V01"  Part="1"
 F 0 "#+3V01" H 2500 5200 50  0001 C CNN
-F 1 "+3V3" V 2375 5225 59  0000 L BNN
+F 1 "+3V3" H 2350 5200 59  0000 L BNN
 F 2 "" H 2500 5200 50  0001 C CNN
 F 3 "" H 2500 5200 50  0001 C CNN
@@
 AR Path="/5B8E25B8/04D4087A" Ref="#+3V3(A)01"  Part="1"
 F 0 "#+3V3(A)01" H 2100 5200 50  0001 C CNN
-F 1 "+3V3(A)" V 1700 5200 59  0000 L BNN
+F 1 "+3V3(A)" H 1925 5200 59  0000 L BNN
 F 2 "" H 2100 5200 50  0001 C CNN
 F 3 "" H 2100 5200 50  0001 C CNN
@@
 AR Path="/5B8E25B8/D7293AB6" Ref="#+3V042"  Part="1"
 F 0 "#+3V042" H 1400 5200 50  0001 C CNN
-F 1 "+3V3" V 1275 5225 59  0000 L BNN
+F 1 "+3V3" H 1275 5200 59  0000 L BNN
 F 2 "" H 1400 5200 50  0001 C CNN
 F 3 "" H 1400 5200 50  0001 C CNN
@@
 AR Path="/5B8E25B8/4FCF2529" Ref="#+3V3(A)02"  Part="1"
 F 0 "#+3V3(A)02" H 8400 2300 50  0001 C CNN
-F 1 "+3V3(A)" V 8000 2275 59  0000 L BNN
+F 1 "+3V3(A)" H 8250 2300 59  0000 L BNN
 F 2 "" H 8400 2300 50  0001 C CNN
 F 3 "" H 8400 2300 50  0001 C CNN
@@
 AR Path="/5B8E25B8/4E54B0A7" Ref="#+3V3(A)03"  Part="1"
 F 0 "#+3V3(A)03" H 8400 3100 50  0001 C CNN
-F 1 "+3V3(A)" V 8000 3100 59  0000 L BNN
+F 1 "+3V3(A)" H 8250 3100 59  0000 L BNN
 F 2 "" H 8400 3100 50  0001 C CNN
 F 3 "" H 8400 3100 50  0001 C CNN
@@
 AR Path="/5B8E25B8/A80C603B" Ref="#+3V010"  Part="1"
 F 0 "#+3V010" H 7400 1000 50  0001 C CNN
-F 1 "+3V3" V 7275 1050 59  0000 L BNN
+F 1 "+3V3" H 7250 1000 59  0000 L BNN
 F 2 "" H 7400 1000 50  0001 C CNN
 F 3 "" H 7400 1000 50  0001 C CNN
@@
 Text Notes 1000 7525 0    42   ~ 0
 More info at http://www.envox.hr/eez
+NoConn ~ 5000 4500
+NoConn ~ 5000 4600
+NoConn ~ 5000 4700
+NoConn ~ 5000 4800
+NoConn ~ 5000 4900
+NoConn ~ 5000 3000
+NoConn ~ 3200 2700
+Text HLabel 1650 4200 0    50   Output ~ 0
+ETH_RXD1
+Text HLabel 1650 4300 0    50   Output ~ 0
+ETH_RXD2
+Text HLabel 1650 4400 0    50   Output ~ 0
+ETH_RXD3
+Text HLabel 1650 4100 0    50   Output ~ 0
+ETH_RXD0
+Text HLabel 1650 4600 0    50   Input ~ 0
+ETH_TXD0
+Text HLabel 1650 4700 0    50   Input ~ 0
+ETH_TXD1
+Text HLabel 1650 4800 0    50   Input ~ 0
+ETH_TXD2
+Text HLabel 1650 4900 0    50   Input ~ 0
+ETH_TXD3
+$Comp
+L power:PWR_FLAG #FLG0101
+U 1 1 5D72DB51
+P 2300 5400
+F 0 "#FLG0101" H 2300 5475 50  0001 C CNN
+F 1 "PWR_FLAG" H 2300 5325 50  0001 C CNN
+F 2 "" H 2300 5400 50  0001 C CNN
+F 3 "~" H 2300 5400 50  0001 C CNN
+	1    2300 5400
+	1    0    0    -1
+$EndComp
+Connection ~ 2300 5400
+Wire Wire Line
+	2300 5400 2100 5400
+Text HLabel 1700 2800 0    50   Output ~ 0
+ETH_RX_DV
+Text HLabel 1700 2700 0    50   Output ~ 0
+ETH_RX_CLK
+Text HLabel 1700 2600 0    50   Input ~ 0
+ETH_TX_EN
+Text HLabel 1700 2500 0    50   Output ~ 0
+ETH_TX_CLK
+Text HLabel 1700 2300 0    50   Input ~ 0
+ETH_MDC
+Text HLabel 1700 2200 0    50   BiDi ~ 0
+ETH_MDIO
+Text HLabel 1700 2000 0    50   Input ~ 0
+MCLK_25
+Text HLabel 1650 3600 0    50   Output ~ 0
+ETH_COL
+Text HLabel 1650 3900 0    50   Output ~ 0
+ETH_CRS
+$Comp
+L EEZ_DIB_MCU_r1B1-eagle-import:C-EUC0603 C64
+U 1 0 B6C25B1D
+P 5800 4700
+AR Path="/B6C25B1D" Ref="C64"  Part="1"
+AR Path="/5B8E25B8/B6C25B1D" Ref="C64"  Part="1"
+F 0 "C64" H 5715 4735 59  0000 R TNN
+F 1 "100n" H 5715 4660 59  0000 R TNN
+F 2 "EEZ DIB MCU r1B1:C0603" H 5800 4700 50  0001 C CNN
+F 3 "" H 5800 4700 50  0001 C CNN
+	1    5800 4700
+	-1   0    0    -1
+$EndComp
+Text GLabel 1650 3800 0    50   Input ~ 0
+~RESET
+Text GLabel 1650 3700 0    50   Output ~ 0
+SPI5_IRQ
 $EndSCHEMATC

Commit message: Updating Kicad Files to r1B2
Some component Values and connections had changed since r1B1 when kicad file was last converted, brought sch and pcb up to current eagle file.
Parts:
- C59, C60, C61, C62, C63, C64, C65, C67, C68, C69, C70: footprint EEZ DIB MCU r1B1:C0603 -> EEZ DIB MCU r1B2:C0603; symbol EEZ_DIB_MCU_r1B1-eagle-import:C-EUC0603 -> EEZ_DIB_MCU_r1B2-eagle-import:C-EUC0603
- C66: footprint EEZ DIB MCU r1B1:EC1206 -> EEZ DIB MCU r1B2:EC1206; symbol EEZ_DIB_MCU_r1B1-eagle-import:ECAP1206 -> EEZ_DIB_MCU_r1B2-eagle-import:ECAP1206
- FB1: value 60R@100MHz -> LCBA-600; footprint EEZ DIB MCU r1B1:BEAD0603 -> EEZ DIB MCU r1B2:BEAD0603; symbol EEZ_DIB_MCU_r1B1-eagle-import:FERRITE_BEAD0603 -> EEZ_DIB_MCU_r1B2-eagle-import:FERRITE_BEAD0603
- IC16: footprint EEZ DIB MCU r1B1:DRL6 -> EEZ DIB MCU r1B2:DRL6; symbol EEZ_DIB_MCU_r1B1-eagle-import:TPD4E001-DRL -> EEZ_DIB_MCU_r1B2-eagle-import:TPD4E001-DRL
- IC17: footprint EEZ DIB MCU r1B1:PT48 -> EEZ DIB MCU r1B2:PT48; symbol EEZ_DIB_MCU_r1B1-eagle-import:DP83848CVV_NOPB -> EEZ_DIB_MCU_r1B2-eagle-import:DP83848CVV_NOPB
- JP5, JP6, JP7, JP8: footprint EEZ DIB MCU r1B1:JP2-CUT -> EEZ DIB MCU r1B2:JP2-CUT; symbol EEZ_DIB_MCU_r1B1-eagle-import:JP2-CUT -> EEZ_DIB_MCU_r1B2-eagle-import:JP2-CUT
- JP9: footprint EEZ DIB MCU r1B1:JP2-NOCUT -> EEZ DIB MCU r1B2:JP2-NOCUT; symbol EEZ_DIB_MCU_r1B1-eagle-import:JP2-NOCUT -> EEZ_DIB_MCU_r1B2-eagle-import:JP2-NOCUT
- R43, R44, R45, R46, R47, R48, R49, R50, R51, R52, R53, R54, R55, R56, R57, R58, R60: footprint EEZ DIB MCU r1B1:R0805 -> EEZ DIB MCU r1B2:R0805; symbol EEZ_DIB_MCU_r1B1-eagle-import:R-EU_R0805 -> EEZ_DIB_MCU_r1B2-eagle-import:R-EU_R0805
- R59: footprint EEZ DIB MCU r1B1:R0603 -> EEZ DIB MCU r1B2:R0603; symbol EEZ_DIB_MCU_r1B1-eagle-import:R-EU_R0603 -> EEZ_DIB_MCU_r1B2-eagle-import:R-EU_R0603
- RN1, RN2, RN3, RN4: footprint EEZ DIB MCU r1B1:CAY16 -> EEZ DIB MCU r1B2:CAY16; symbol EEZ_DIB_MCU_r1B1-eagle-import:R_ARRAY4 -> EEZ_DIB_MCU_r1B2-eagle-import:R_ARRAY4
- SPEED: value HSMY-C170 -> LTST-C170YKT; footprint EEZ DIB MCU r1B1:LED_0805 -> EEZ DIB MCU r1B2:LED_0805; symbol EEZ_DIB_MCU_r1B1-eagle-import:LED0805 -> EEZ_DIB_MCU_r1B2-eagle-import:LED0805
- X6: footprint EEZ DIB MCU r1B1:RJ45-TRAFO-LED -> EEZ DIB MCU r1B2:RJ45-TRAFO-LED; symbol EEZ_DIB_MCU_r1B1-eagle-import:RJ45-TRAFO-LED -> EEZ_DIB_MCU_r1B2-eagle-import:RJ45-TRAFO-LED
Connections:
- net labels added: ETH_RX+, ETH_RX-, ETH_TX+, ETH_TX-

Commit message: Updating Kicad Files To Reflect Latest Commits
Changed lines of the file:
@@
 Wire Wire Line
 	2600 3500 2500 3500
-Text GLabel 2600 3500 0    10   BiDi ~ 0
-+3V3
 Wire Wire Line
 	5400 5000 5400 4900
@@
 Wire Wire Line
 	3100 1600 3100 1700
-Text GLabel 3100 1600 0    10   BiDi ~ 0
-+3V3
 Wire Wire Line
 	2000 5000 2200 5000
-Text GLabel 2000 5000 0    10   BiDi ~ 0
-+3V3
 Wire Wire Line
 	7600 1200 7400 1200
@@
 AR Path="/8BD298C6" Ref="SPEED"  Part="1"
 AR Path="/5B8E25B8/8BD298C6" Ref="SPEED1"  Part="1"
-F 0 "SPEED1" V 6040 3270 59  0000 L BNN
-F 1 "LTST-C170YKT" V 5775 3120 59  0000 L BNN
+F 0 "SPEED1" V 5975 3000 59  0000 L BNN
+F 1 "LTST-C170YKT" V 6075 3000 59  0000 L BNN
 F 2 "EEZ DIB MCU r1B2:LED_0805" H 5900 3300 50  0001 C CNN
 F 3 "" H 5900 3300 50  0001 C CNN
@@
 AR Path="/5B8E25B8/DB1F9C9B" Ref="#+3V043"  Part="1"
 F 0 "#+3V043" H 6800 2900 50  0001 C CNN
-F 1 "+3V3" V 6525 2875 59  0000 L BNN
+F 1 "+3V3" H 6625 2900 59  0000 L BNN
 F 2 "" H 6800 2900 50  0001 C CNN
 F 3 "" H 6800 2900 50  0001 C CNN
@@
 AR Path="/5B8E25B8/29960DDB" Ref="RN2"  Part="4"
 F 0 "RN2" H 2200 3705 59  0000 R BNN
-F 1 "DR1206-33R-4/8" H 2600 3705 59  0000 L BNN
+F 1 "DR1206-33R-4/8" H 2275 3375 59  0000 L BNN
 F 2 "EEZ DIB MCU r1B2:CAY16" H 2400 3700 50  0001 C CNN
 F 3 "" H 2400 3700 50  0001 C CNN
@@
 AR Path="/5B8E25B8/E3F447F6" Ref="RN4"  Part="4"
 F 0 "RN4" H 2200 4605 59  0000 R BNN
-F 1 "DR1206-33R-4/8" H 2600 4605 59  0000 L BNN
+F 1 "DR1206-33R-4/8" H 2300 4075 59  0000 L BNN
 F 2 "EEZ DIB MCU r1B2:CAY16" H 2400 4600 50  0001 C CNN
 F 3 "" H 2400 4600 50  0001 C CNN
@@
 AR Path="/5B8E25B8/107F392D" Ref="RN1"  Part="4"
 F 0 "RN1" H 2000 2005 59  0000 R BNN
-F 1 "DR1206-33R-4/8" H 2400 2005 59  0000 L BNN
+F 1 "DR1206-33R-4/8" H 2075 2050 59  0000 L BNN
 F 2 "EEZ DIB MCU r1B2:CAY16" H 2200 2000 50  0001 C CNN
 F 3 "" H 2200 2000 50  0001 C CNN
@@
 AR Path="/5B8E25B8/EB5F8C4A" Ref="#+3V03"  Part="1"
 F 0 "#+3V03" H 3100 1500 50  0001 C CNN
-F 1 "+3V3" V 3150 1475 59  0000 L BNN
+F 1 "+3V3" H 2975 1525 59  0000 L BNN
 F 2 "" H 3100 1500 50  0001 C CNN
 F 3 "" H 3100 1500 50  0001 C CNN
@@
 AR Path="/5B8E25B8/490C85BF" Ref="RN3"  Part="4"
 F 0 "RN3" H 2200 4305 59  0000 R BNN
-F 1 "DR1206-33R-4/8" H 2600 4305 59  0000 L BNN
+F 1 "DR1206-33R-4/8" H 2300 4100 59  0000 L BNN
 F 2 "EEZ DIB MCU r1B2:CAY16" H 2400 4300 50  0001 C CNN
 F 3 "" H 2400 4300 50  0001 C CNN
@@
 AR Path="/357D3C8D" Ref="JP8"  Part="1"
 AR Path="/5B8E25B8/357D3C8D" Ref="JP8"  Part="1"
-F 0 "JP8" H 1925 3600 59  0000 R BNN
+F 0 "JP8" H 1925 3725 59  0000 R BNN
 F 1 "JP2-CUT" H 1800 3700 50  0001 C CNN
 F 2 "EEZ DIB MCU r1B2:JP2-CUT" H 1800 3700 50  0001 C CNN
