File: mcu/KiCad/SDRAM,_JTAG,_SD_card,_EEPROM.sch (KiCad schematic (older format))
At the start: 26 parts, among them IC6 TPD4E001DRLR, IC7 TPD4E001DRLR, IC8 IS42S16400J, IC9 BR24G64FVT-3AGE2, J1 5033981892, X4 ZL231-20KG

Commit message: Kicad-ised schematic, fixed import errors
Basic stuff like pin functions not assigned, and moving to heirarchial labels instead of global,
Connections:
- wire segments 204 -> 201
- no-connect marks 0 -> 6

Commit message: Updating Kicad Files to r1B2
Some component Values and connections had changed since r1B1 when kicad file was last converted, brought sch and pcb up to current eagle file.
Parts:
- C35, C36, C38, C39, C40, C41, C42, C43, C44: footprint EEZ DIB MCU r1B1:C0603 -> EEZ DIB MCU r1B2:C0603; symbol EEZ_DIB_MCU_r1B1-eagle-import:C-EUC0603 -> EEZ_DIB_MCU_r1B2-eagle-import:C-EUC0603
- C37: footprint EEZ DIB MCU r1B1:C1210 -> EEZ DIB MCU r1B2:C1206; symbol EEZ_DIB_MCU_r1B1-eagle-import:C-EUC1210 -> EEZ_DIB_MCU_r1B2-eagle-import:C-EUC1210
- IC6, IC7: footprint EEZ DIB MCU r1B1:DRL6 -> EEZ DIB MCU r1B2:DRL6; symbol EEZ_DIB_MCU_r1B1-eagle-import:TPD4E001-DRL -> EEZ_DIB_MCU_r1B2-eagle-import:TPD4E001-DRL
- IC8: footprint EEZ DIB MCU r1B1:TSOPII-54 -> EEZ DIB MCU r1B2:TSOPII-54; symbol EEZ_DIB_MCU_r1B1-eagle-import:IS42S16400 -> EEZ_DIB_MCU_r1B2-eagle-import:IS42S16400
- IC9: footprint EEZ DIB MCU r1B1:PW8_TSSOP8 -> EEZ DIB MCU r1B2:PW8_TSSOP8; symbol EEZ_DIB_MCU_r1B1-eagle-import:BR24GXXX-TSSOP -> EEZ_DIB_MCU_r1B2-eagle-import:BR24GXXX-TSSOP
- J1: value 5033981892 -> 503398-1892; footprint EEZ DIB MCU r1B1:5033981892 -> EEZ DIB MCU r1B2:5033981892; symbol EEZ_DIB_MCU_r1B1-eagle-import:5033981892 -> EEZ_DIB_MCU_r1B2-eagle-import:5033981892
- JP3: footprint EEZ DIB MCU r1B1:JP2-NOCUT -> EEZ DIB MCU r1B2:JP2-NOCUT; symbol EEZ_DIB_MCU_r1B1-eagle-import:JP2-NOCUT -> EEZ_DIB_MCU_r1B2-eagle-import:JP2-NOCUT
- R19, R20, R21, R22, R23, R24, R25, R26, R27: footprint EEZ DIB MCU r1B1:R0805 -> EEZ DIB MCU r1B2:R0805; symbol EEZ_DIB_MCU_r1B1-eagle-import:R-EU_R0805 -> EEZ_DIB_MCU_r1B2-eagle-import:R-EU_R0805
- X4: footprint EEZ DIB MCU r1B1:ML20L -> EEZ DIB MCU r1B2:ML20L; symbol EEZ_DIB_MCU_r1B1-eagle-import:IDC-20PIN-ANGLED -> EEZ_DIB_MCU_r1B2-eagle-import:IDC-20PIN-ANGLED

Commit message: Updating Kicad Files To Reflect Latest Commits
Parts:
- C37: value 10u -> 4u7
Changed lines of the file:
@@
 AR Path="/5B8E1D28/59F31A24" Ref="#+3V034"  Part="1"
 F 0 "#+3V034" H 2300 5500 50  0001 C CNN
-F 1 "+3V3" H 1975 5425 59  0000 L BNN
+F 1 "+3V3" H 2150 5525 59  0000 L BNN
 F 2 "" H 2300 5500 50  0001 C CNN
 F 3 "" H 2300 5500 50  0001 C CNN
@@
 AR Path="/5B8E1D28/CDD0F144" Ref="#+3V0312"  Part="1"
 F 0 "#+3V0312" H 9700 4100 50  0001 C CNN
-F 1 "+3V3" V 9575 4125 59  0000 L BNN
+F 1 "+3V3" H 9550 4125 59  0000 L BNN
 F 2 "" H 9700 4100 50  0001 C CNN
 F 3 "" H 9700 4100 50  0001 C CNN
@@
 AR Path="/5B8E1D28/DB614CD6" Ref="C37"  Part="1"
 F 0 "C37" V 9481 4505 59  0000 R BNN
-F 1 "10u" V 9581 4505 59  0000 R BNN
+F 1 "4u7" V 9581 4505 59  0000 R BNN
 F 2 "EEZ DIB MCU r1B2:C1206" H 9500 4600 50  0001 C CNN
 F 3 "" H 9500 4600 50  0001 C CNN
