File: mcu/KiCad/STM32F7_MCU.sch (KiCad schematic (older format))
At the start: 45 parts, among them IC4 STM32F769IGT6, IC5 LD1117ADT33TR, Y1 10MHz

Commit message: Kicad-ised schematic, fixed import errors
Basic stuff like pin functions not assigned, and moving to heirarchial labels instead of global,
Connections:
- net labels added: LTDC_B[2..7], LTDC_G[2..7], LTDC_R[2..7]
- wire segments 302 -> 304
- no-connect marks 0 -> 6

Commit message: Updating Kicad Files to r1B2
Some component Values and connections had changed since r1B1 when kicad file was last converted, brought sch and pcb up to current eagle file.
Parts:
- B1: footprint EEZ DIB MCU r1B1:DS1092-16-B6P -> EEZ DIB MCU r1B2:DS1092-16-B6P; symbol EEZ_DIB_MCU_r1B1-eagle-import:CELL_BATTERY-THT20MM -> EEZ_DIB_MCU_r1B2-eagle-import:CELL_BATTERY-THT20MM
- C10: value 47u -> EEEFK1V470P; footprint EEZ DIB MCU r1B1:CAPAE660X610N -> EEZ DIB MCU r1B2:CAPAE660X610N; symbol EEZ_DIB_MCU_r1B1-eagle-import:ECAPPANASONIC_H -> EEZ_DIB_MCU_r1B2-eagle-import:ECAPPANASONIC_H
- C11, C13, C14, C15, C16, C17, C18, C20, C22, C23, C24, C25, C26, C27, C28, C29, C32, C8, C9: footprint EEZ DIB MCU r1B1:C0603 -> EEZ DIB MCU r1B2:C0603; symbol EEZ_DIB_MCU_r1B1-eagle-import:C-EUC0603 -> EEZ_DIB_MCU_r1B2-eagle-import:C-EUC0603
- C12: value 10u -> 4u7; footprint EEZ DIB MCU r1B1:EC1206 -> EEZ DIB MCU r1B2:EC1206; symbol EEZ_DIB_MCU_r1B1-eagle-import:ECAP1206 -> EEZ_DIB_MCU_r1B2-eagle-import:ECAP1206
- C19: footprint EEZ DIB MCU r1B1:EC1206 -> EEZ DIB MCU r1B2:EC1206; symbol EEZ_DIB_MCU_r1B1-eagle-import:ECAP1206 -> EEZ_DIB_MCU_r1B2-eagle-import:ECAP1206
- C21, C30, C31, C33, C34: footprint EEZ DIB MCU r1B1:C0805 -> EEZ DIB MCU r1B2:C0805; symbol EEZ_DIB_MCU_r1B1-eagle-import:C-EUC0805 -> EEZ_DIB_MCU_r1B2-eagle-import:C-EUC0805
- D1: footprint EEZ DIB MCU r1B1:DO214AA -> EEZ DIB MCU r1B2:DO214AA; symbol EEZ_DIB_MCU_r1B1-eagle-import:DIODEDO214AA -> EEZ_DIB_MCU_r1B2-eagle-import:DIODEDO214AA
- FM1, FM2: footprint EEZ DIB MCU r1B1:FIDUCIAL -> EEZ DIB MCU r1B2:FIDUCIAL; symbol EEZ_DIB_MCU_r1B1-eagle-import:FIDUCIAL -> EEZ_DIB_MCU_r1B2-eagle-import:FIDUCIAL
- IC4: footprint EEZ DIB MCU r1B1:LQFP-176_24X24MM -> EEZ DIB MCU r1B2:LQFP-176_24X24MM; symbol EEZ_DIB_MCU_r1B1-eagle-import:STM32F769IXT -> EEZ_DIB_MCU_r1B2-eagle-import:STM32F769IXT
- IC5: footprint EEZ DIB MCU r1B1:DPACK -> EEZ DIB MCU r1B2:DPACK; symbol EEZ_DIB_MCU_r1B1-eagle-import:LD117A?DT -> EEZ_DIB_MCU_r1B2-eagle-import:LD117A?DT
- JP1, JP2: footprint EEZ DIB MCU r1B1:JP3-CUT -> EEZ DIB MCU r1B2:JP3-CUT; symbol EEZ_DIB_MCU_r1B1-eagle-import:JP3-CUT -> EEZ_DIB_MCU_r1B2-eagle-import:JP3-CUT
- L1: footprint EEZ DIB MCU r1B1:BEAD0603 -> EEZ DIB MCU r1B2:BEAD0603; symbol EEZ_DIB_MCU_r1B1-eagle-import:FERRITE_BEAD0603 -> EEZ_DIB_MCU_r1B2-eagle-import:FERRITE_BEAD0603
- R11, R12, R13, R14, R15, R16, R17, R18: footprint EEZ DIB MCU r1B1:R0805 -> EEZ DIB MCU r1B2:R0805; symbol EEZ_DIB_MCU_r1B1-eagle-import:R-EU_R0805 -> EEZ_DIB_MCU_r1B2-eagle-import:R-EU_R0805
- Y1: footprint EEZ DIB MCU r1B1:HC-49_4H -> EEZ DIB MCU r1B2:HC-49_4H; symbol EEZ_DIB_MCU_r1B1-eagle-import:XTALSMD -> EEZ_DIB_MCU_r1B2-eagle-import:XTALSMD

Commit message: Updating Kicad Files To Reflect Latest Commits
Changed lines of the file:
@@
 Text Label 2400 2200 0    50   ~ 0
 LTDC_R[2..7],LTDC_G[2..7],LTDC_B[2..7]
-Text Label 6250 2200 1    50   ~ 0
+Text Label 7525 2200 2    50   ~ 0
 LTDC_R[2..7],LTDC_G[2..7],LTDC_B[2..7]
 Wire Wire Line
@@
 Wire Wire Line
 	10700 3000 10600 3000
-Text Label 10600 2700 2    50   ~ 0
+Text Label 10275 2700 2    50   ~ 0
 BOOT0
 Wire Wire Line
@@
 Wire Wire Line
 	4100 8500 4000 8500
-Text Label 4100 8500 2    50   ~ 0
+Text Label 4000 8500 2    50   ~ 0
 VREF+
 Wire Wire Line
@@
 AR Path="/5B8E1886/B7CA437E" Ref="#+3V033"  Part="1"
 F 0 "#+3V033" H 10800 6100 50  0001 C CNN
-F 1 "+3V3" V 10675 6150 59  0000 L BNN
+F 1 "+3V3" H 10700 6125 59  0000 L BNN
 F 2 "" H 10800 6100 50  0001 C CNN
 F 3 "" H 10800 6100 50  0001 C CNN
@@
 AR Path="/5B8E1886/34CFF32A" Ref="#+3V012"  Part="1"
 F 0 "#+3V012" H 1400 3900 50  0001 C CNN
-F 1 "+3V3" V 1450 3875 59  0000 L BNN
+F 1 "+3V3" H 1300 3950 59  0000 L BNN
 F 2 "" H 1400 3900 50  0001 C CNN
 F 3 "" H 1400 3900 50  0001 C CNN
@@
 AR Path="/5B8E1886/04853D9A" Ref="#+3V014"  Part="1"
 F 0 "#+3V014" H 1300 5800 50  0001 C CNN
-F 1 "+3V3" V 1325 5775 59  0000 L BNN
+F 1 "+3V3" H 1175 5850 59  0000 L BNN
 F 2 "" H 1300 5800 50  0001 C CNN
 F 3 "" H 1300 5800 50  0001 C CNN
