File: mcu/KiCad/TFT,_Audio,_USB.sch (KiCad schematic (older format))
At the start: 45 parts, among them IC10 TPS2051BDBVR, IC11 TPS61169DCKR, IC12 TPD4E001DRLR, IC13 TPA6205A1DGN, IC14 TPD4E001DRLR, IC15 AR1021-I/SS, Q1 MMBT5551, X5 292304-1

Commit message: Kicad-ised schematic, fixed import errors
Basic stuff like pin functions not assigned, and moving to heirarchial labels instead of global,
Connections:
- net labels added: LTDC_B[2..7], LTDC_G[2..7], LTDC_R[2..7]
- wire segments 214 -> 213
- no-connect marks 0 -> 3

Commit message: Updating Kicad Files to r1B2
Some component Values and connections had changed since r1B1 when kicad file was last converted, brought sch and pcb up to current eagle file.
Parts:
- removed X5: 292304-1, EEZ DIB MCU r1B1:USB-B, symbol EEZ_DIB_MCU_r1B1-eagle-import:USB-B292304-1
- added J2: 67803-8020, EEZ DIB MCU r1B2:678038020, symbol EEZ_DIB_MCU_r1B2-eagle-import:678038020
- C45: footprint EEZ DIB MCU r1B1:C1206 -> EEZ DIB MCU r1B2:C1206; symbol EEZ_DIB_MCU_r1B1-eagle-import:C-EUC1206 -> EEZ_DIB_MCU_r1B2-eagle-import:C-EUC1206
- C46, C48, C50, C51, C52, C54, C57, C58: footprint EEZ DIB MCU r1B1:C0805 -> EEZ DIB MCU r1B2:C0805; symbol EEZ_DIB_MCU_r1B1-eagle-import:C-EUC0805 -> EEZ_DIB_MCU_r1B2-eagle-import:C-EUC0805
- C47: value 4u7/16V (293D475X9016A2TE3) -> 4u7; footprint EEZ DIB MCU r1B1:EC1206 -> EEZ DIB MCU r1B2:EC1206; symbol EEZ_DIB_MCU_r1B1-eagle-import:ECAP1206 -> EEZ_DIB_MCU_r1B2-eagle-import:ECAP1206
- C49, C53, C55: footprint EEZ DIB MCU r1B1:C0603 -> EEZ DIB MCU r1B2:C0603; symbol EEZ_DIB_MCU_r1B1-eagle-import:C-EUC0603 -> EEZ_DIB_MCU_r1B2-eagle-import:C-EUC0603
- C56: value 220n -> 470n; footprint EEZ DIB MCU r1B1:C0805 -> EEZ DIB MCU r1B2:C0805; symbol EEZ_DIB_MCU_r1B1-eagle-import:C-EUC0805 -> EEZ_DIB_MCU_r1B2-eagle-import:C-EUC0805
- D2: value NSR0240 -> RB751V40T1G or NSR0240; footprint EEZ DIB MCU r1B1:SOD123 -> EEZ DIB MCU r1B2:SOD123; symbol EEZ_DIB_MCU_r1B1-eagle-import:SCHOTTKYSOD123 -> EEZ_DIB_MCU_r1B2-eagle-import:SCHOTTKYSOD123
- IC10: footprint EEZ DIB MCU r1B1:DBV5 -> EEZ DIB MCU r1B2:DBV5; symbol EEZ_DIB_MCU_r1B1-eagle-import:TPS2051B -> EEZ_DIB_MCU_r1B2-eagle-import:TPS2051B
- IC11: footprint EEZ DIB MCU r1B1:DCK5 -> EEZ DIB MCU r1B2:DCK5; symbol EEZ_DIB_MCU_r1B1-eagle-import:TPS61169DCKR -> EEZ_DIB_MCU_r1B2-eagle-import:TPS61169DCKR
- IC12, IC14: footprint EEZ DIB MCU r1B1:DRL6 -> EEZ DIB MCU r1B2:DRL6; symbol EEZ_DIB_MCU_r1B1-eagle-import:TPD4E001-DRL -> EEZ_DIB_MCU_r1B2-eagle-import:TPD4E001-DRL
- IC13: footprint EEZ DIB MCU r1B1:SOP65P490X110-9N -> EEZ DIB MCU r1B2:SOP65P490X110-9N; symbol EEZ_DIB_MCU_r1B1-eagle-import:TPA6205 -> EEZ_DIB_MCU_r1B2-eagle-import:TPA6205
- IC15: footprint EEZ DIB MCU r1B1:SOP65P780X200-20N -> EEZ DIB MCU r1B2:SOP65P780X200-20N; symbol EEZ_DIB_MCU_r1B1-eagle-import:AR1021-I_SS -> EEZ_DIB_MCU_r1B2-eagle-import:AR1021-I_SS
- JP4: footprint EEZ DIB MCU r1B1:JP3-CUT -> EEZ DIB MCU r1B2:JP3-CUT; symbol EEZ_DIB_MCU_r1B1-eagle-import:JP3-CUT -> EEZ_DIB_MCU_r1B2-eagle-import:JP3-CUT
- L2: footprint EEZ DIB MCU r1B1:DE0403 -> EEZ DIB MCU r1B2:DE0403; symbol EEZ_DIB_MCU_r1B1-eagle-import:DE0403 -> EEZ_DIB_MCU_r1B2-eagle-import:DE0403
- LCD1: footprint EEZ DIB MCU r1B1:FPC_40 -> EEZ DIB MCU r1B2:FPC_40; symbol EEZ_DIB_MCU_r1B1-eagle-import:RFE430Y-AIW-DNS -> EEZ_DIB_MCU_r1B2-eagle-import:RFE430Y-AIW-DNS
- Q1: footprint EEZ DIB MCU r1B1:SOT23-BEC -> EEZ DIB MCU r1B2:SOT23-BEC; symbol EEZ_DIB_MCU_r1B1-eagle-import:-NPN-SOT23-BEC -> EEZ_DIB_MCU_r1B2-eagle-import:-NPN-SOT23-BEC
- R28, R29, R30, R31, R32, R33, R34, R35, R36, R37, R38, R39, R40, R41, R42: footprint EEZ DIB MCU r1B1:R0805 -> EEZ DIB MCU r1B2:R0805; symbol EEZ_DIB_MCU_r1B1-eagle-import:R-EU_R0805 -> EEZ_DIB_MCU_r1B2-eagle-import:R-EU_R0805
- SP1: footprint EEZ DIB MCU r1B1:LD-BZEL-M1313 -> EEZ DIB MCU r1B2:LD-BZEL-M1313; symbol EEZ_DIB_MCU_r1B1-eagle-import:LD-BZEL-M1313 -> EEZ_DIB_MCU_r1B2-eagle-import:LD-BZEL-M1313
- TOUCH, VBUS: footprint EEZ DIB MCU r1B1:LED_0805 -> EEZ DIB MCU r1B2:LED_0805; symbol EEZ_DIB_MCU_r1B1-eagle-import:LED0805 -> EEZ_DIB_MCU_r1B2-eagle-import:LED0805
- ZD3: footprint EEZ DIB MCU r1B1:SOD323-W -> EEZ DIB MCU r1B2:SOD323-W; symbol EEZ_DIB_MCU_r1B1-eagle-import:ZENER-DIODESOD323 -> EEZ_DIB_MCU_r1B2-eagle-import:ZENER-DIODESOD323
Connections:
- net labels added: LTDC_RESET, SPKR+, SPKR-, Touch_XL, Touch_XR, Touch_YD, Touch_YU, VLED_SW
- wire segments 213 -> 219
- no-connect marks 3 -> 2

Commit message: Updating Kicad Files To Reflect Latest Commits
Parts:
- D2: footprint EEZ DIB MCU r1B2:SOD123 -> EEZ DIB MCU r1B2:SOD323-R
Changed lines of the file:
@@
 AR Path="/5B8E2134/873B455E" Ref="#+3V0317"  Part="1"
 F 0 "#+3V0317" H 6400 5000 50  0001 C CNN
-F 1 "+3V3" V 6475 5025 59  0000 L TNN
+F 1 "+3V3" H 6275 5075 59  0000 L TNN
 F 2 "" H 6400 5000 50  0001 C CNN
 F 3 "" H 6400 5000 50  0001 C CNN
@@
 AR Path="/5B8E2134/4B764152" Ref="#+3V0316"  Part="1"
 F 0 "#+3V0316" H 4100 2100 50  0001 C CNN
-F 1 "+3V3" V 4225 2200 59  0000 R TNN
+F 1 "+3V3" H 4275 2175 59  0000 R TNN
 F 2 "" H 4100 2100 50  0001 C CNN
 F 3 "" H 4100 2100 50  0001 C CNN
@@
 F 0 "D2" H 3550 1375 59  0000 R BNN
 F 1 "RB751V40T1G or NSR0240" H 4175 1275 59  0000 R BNN
-F 2 "EEZ DIB MCU r1B2:SOD123" H 3500 1200 50  0001 C CNN
+F 2 "EEZ DIB MCU r1B2:SOD323-R" H 3500 1200 50  0001 C CNN
 F 3 "" H 3500 1200 50  0001 C CNN
 	1    3500 1200
@@
 AR Path="/5B8E2134/5569F9BF" Ref="#+3V0314"  Part="1"
 F 0 "#+3V0314" H 2400 5300 50  0001 C CNN
-F 1 "+3V3" V 2275 5325 59  0000 L BNN
+F 1 "+3V3" H 2325 5325 59  0000 L BNN
 F 2 "" H 2400 5300 50  0001 C CNN
 F 3 "" H 2400 5300 50  0001 C CNN
@@
 AR Path="/5B8E2134/85BCDC48" Ref="#+3V0318"  Part="1"
 F 0 "#+3V0318" H 8900 4300 50  0001 C CNN
-F 1 "+3V3" V 8775 4325 59  0000 L BNN
+F 1 "+3V3" H 8800 4325 59  0000 L BNN
 F 2 "" H 8900 4300 50  0001 C CNN
 F 3 "" H 8900 4300 50  0001 C CNN
@@
 AR Path="/5B8E2134/48C2C5DB" Ref="#P+03"  Part="1"
 F 0 "#P+03" H 7900 1400 50  0001 C CNN
-F 1 "+5V" V 7950 1375 59  0000 L BNN
+F 1 "+5V" H 7825 1400 59  0000 L BNN
 F 2 "" H 7900 1400 50  0001 C CNN
 F 3 "" H 7900 1400 50  0001 C CNN
@@
 AR Path="/5B8E2134/459FCD94" Ref="#P+04"  Part="1"
 F 0 "#P+04" H 10600 1000 50  0001 C CNN
-F 1 "+5V" V 10650 975 59  0000 L BNN
+F 1 "+5V" H 10575 1025 59  0000 L BNN
 F 2 "" H 10600 1000 50  0001 C CNN
 F 3 "" H 10600 1000 50  0001 C CNN
@@
 Wire Wire Line
 	9700 3600 9700 2900
+Connection ~ 9700 2900
+Wire Wire Line
+	9700 2900 10600 2900
 Wire Bus Line
 	6475 2800 6475 3300
@@
 Wire Bus Line
 	6475 2000 6475 2500
-Connection ~ 9700 2900
-Wire Wire Line
-	9700 2900 10600 2900
 $EndSCHEMATC
