File: mcu/Eagle files/EEZ DIB MCU r1B2.sch (EAGLE design)
At the start: 190 parts, among them IC1 TPD4E001DRLR, IC10 TPS2051BDBVR, IC11 TPS61169DCKR, IC12 TPD4E001DRLR, IC13 TPA6205A1DGN, IC14 TPD4E001DRLR, IC15 AR1021-I/SS, IC16 TPD4E001DRLR, IC17 DP83848CVV/NOPB, IC2 SN74LVC2G34DBVR, IC3 BTS3408G, IC4 STM32F769IGT6, IC5 LD1117ADT33TR, IC6 TPD4E001DRLR, IC7 TPD4E001DRLR, IC8 IS42S16400J, IC9 AT24C02D-SSHM-T, J1 503398-1892, J2 67803-8020, Q1 MMBT5551, SW1 PEC16-2215F-S0024, SW2 TL1100CF160Q, X1 ZL263-40DG, X2 ZL231-16KG, X3 1844249, X4 ZL231-20KG, X5 LMJTAB881243M-L, Y1 25MHz

Commit message: #11
Parts:
- removed C70: 100n, rcl:C-EUC0603
- removed IC17: DP83848CVV/NOPB, EEZ_Lib1:DP83848CVV/NOPB
- removed R58, R60: 2K2, rcl:R-EU_R0805
- removed R59: 4K87, rcl:R-EU_R0805
- C36, C44: value 100n -> 4u7; device rcl:C-EUC0603 -> rcl:C-EUC1206
- C37: value 4u7 -> 100n; device rcl:C-EUC1206 -> rcl:C-EUC0603
- C45: value 4u7 -> 1u; device rcl:C-EUC1206 -> rcl:C-EUC0805
- C46: value 1u -> 4u7; device rcl:C-EUC0805 -> EEZ_Lib1:ECAP1206
- C47: value 4u7 -> 2u2; device EEZ_Lib1:ECAP1206 -> rcl:C-EUC0805
- C48: value 2u2 -> 100n; device rcl:C-EUC0805 -> rcl:C-EUC0603
- C49, C53: value 100n -> 1u; device rcl:C-EUC0603 -> rcl:C-EUC0805
- C50: value 1u -> 470n
- C52: value 470n -> 100n; device rcl:C-EUC0805 -> rcl:C-EUC0603
- C54: value 1u -> 100n; device rcl:C-EUC0805 -> rcl:C-EUC0603
- C55: value 100n -> 470n; device rcl:C-EUC0603 -> rcl:C-EUC0805
- C56: value 470n -> 10n
- C58: value 10n -> 100n; device rcl:C-EUC0805 -> rcl:C-EUC0603
- C65: value 100n -> 10u; device rcl:C-EUC0603 -> EEZ_Lib1:ECAP1206
- C66: value 10u -> 100n; device EEZ_Lib1:ECAP1206 -> rcl:C-EUC0603
- IC10: value TPS2051BDBVR -> TPS61169DCKR; device EEZ_Lib1:TPS2051B -> EEZ_Lib1:TPS61169DCKR
- IC11: value TPS61169DCKR -> TPD4E001DRLR; device EEZ_Lib1:TPS61169DCKR -> EEZ_Lib1:TPD4E001-DRL
- IC12: value TPD4E001DRLR -> TPA6205A1DGN; device EEZ_Lib1:TPD4E001-DRL -> EEZ_Lib1:TPA6205
- IC13: value TPA6205A1DGN -> TPD4E001DRLR; device EEZ_Lib1:TPA6205 -> EEZ_Lib1:TPD4E001-DRL
- IC14: value TPD4E001DRLR -> AR1021-I/SS; device EEZ_Lib1:TPD4E001-DRL -> EEZ_Lib1:AR1021-I/SS
- IC15: value AR1021-I/SS -> TPD4E001DRLR; device EEZ_Lib1:AR1021-I/SS -> EEZ_Lib1:TPD4E001-DRL
- IC16: value TPD4E001DRLR -> DP83848CVV/NOPB; device EEZ_Lib1:TPD4E001-DRL -> EEZ_Lib1:DP83848CVV/NOPB
- IC7: value TPD4E001DRLR -> IS42S16400J; device EEZ_Lib1:TPD4E001-DRL -> EEZ_Lib1:IS42S16400
- IC8: value IS42S16400J -> AT24C02D-SSHM-T; device EEZ_Lib1:IS42S16400 -> EEZ_Lib1:AT24CXXSOIC8
- IC9: value AT24C02D-SSHM-T -> TPS2051BDBVR; device EEZ_Lib1:AT24CXXSOIC8 -> EEZ_Lib1:TPS2051B
- JP3: value JP2-NOCUT -> JP2-CUT; device EEZ_Lib1:JP2-NOCUT -> EEZ_Lib1:JP2-CUT
- JP8: value JP2-CUT -> JP2-NOCUT; device EEZ_Lib1:JP2-CUT -> EEZ_Lib1:JP2-NOCUT
- R19, R32: value 47K -> 10K
- R22, R23, R37: value 10K -> 47K
- R25: value 10K -> 10R
- R26: value 47K -> 220R
- R27: value 47K -> 10R
- R28: value 10R -> 47K
- R29: value 220R -> 47K
- R30: value 10R -> 22R
- R31: value 47K -> 22R
- R33: value 22R -> 20K
- R34: value 22R -> 10K
- R38: value 10K -> 20K
- R39: value 20K -> 4K7
- R40: value 47K -> 1K5
- R41: value 20K -> 49R9
- R42: value 4K7 -> 49R9
- R43: value 1K5 -> 2K2
- R44, R48: value 49R9 -> 2K2
- R47, R52: value 2K2 -> 220R
- R50: value 220R -> 49R9
- R53: value 49R9 -> 220R
- R55: value 220R -> 2K2
- R56: value 220R -> 4K87
- SW1: value PEC16-2215F-S0024 -> TL1100CF160Q; device EEZ_switches:ENCODER_SW-PEC16 -> EEZ_switches:TL1100C
- SW2: value TL1100CF160Q -> PEC16-2215F-S0024; device EEZ_switches:TL1100C -> EEZ_switches:ENCODER_SW-PEC16
- X4: value ZL231-20KG -> 22-23-2061; device EEZ_connectors:IDC-20PIN-ANGLED -> EEZ_connectors:22-23-2061
Connections:
- removed net DBGACK: R24.1, X4-19.1
- removed net DBGRQ: R23.1, X4-17.1
- removed net RTCK: R22.1, X4-11.1
- removed net SYS_JTDI: IC4A.PA15, IC6.IO4, X4-5.1
- removed net SYS_JTRST: IC4A.PB4, JP3.1, R19.2
- removed net TRST: IC6.IO1, JP3.2, X4-3.1
- new net ETH_RX_ERR: IC4A.PB10, JP8.2
- new net N$51: JP3.2, R19.2, X4-1.S
- net !AUDIO_SHDN: now also IC12.!SHDN, R37.1; no longer IC13.!SHDN, R40.1
- net !RESET: now also IC16.RESET_N, IC6.IO3, X4-5.S; no longer IC17.RESET_N, IC7.IO3, X4-15.1
- net !USB_OTG_FS_OC: now also IC9.!OC, R28.1; no longer IC10.!OC, R31.1
- net +3V3: now also C37.2, C38.1, C47.1, C49.2, C52.2, C58.1, C68.1, IC12.VDD, IC13.VCC, IC14.VDD, IC15.VCC, IC16.IOVDD33-32, IC16.IOVDD33-48, IC7.VDD-1, IC7.VDD-14, IC7.VDD-27, IC7.VDDQ-3, IC7.VDDQ-43, IC7.VDDQ-49, IC7.VDDQ-9, IC8.VCC, JP3.1, R22.1, R23.1, R24.1, R28.2, R32.2, R37.2, R44.1, R48.1, R49.1, R55.1; no longer C37.1, C38.2, C44.1, C48.1, C50.2, C55.2, C59.1, C70.1, IC13.VDD, IC14.VCC, IC15.VDD, IC16.VCC, IC17.IOVDD33-32, IC17.IOVDD33-48, IC7.VCC, IC8.VDD-1, IC8.VDD-14, IC8.VDD-27, IC8.VDDQ-3, IC8.VDDQ-43, IC8.VDDQ-49, IC8.VDDQ-9, IC9.VCC, R19.1, R25.1, R26.1, R27.1, R31.2, R35.2, R43.2, R50.1, R52.1, R58.1, R60.1, X4-1.1, X4-2.1
- net +3V3(A): now also C60.2, C62.2, C67.1, IC16.AVDD33; no longer C61.2, C63.2, C68.1, IC17.AVDD33
- net +5V: now also C44.1, IC9.IN, R25.1; no longer C45.1, IC10.IN, R28.1
- net DAC_OUT1: now also C51.2; no longer C52.2
- net ENC_SW: now also SW2-2.2; no longer SW1-2.2
- net EOUT_A: now also SW2-1.B; no longer SW1-1.B
- net EOUT_B: now also SW2-1.A; no longer SW1-1.A
- net ETH_MDC: now also IC16.MDC; no longer IC17.MDC
- net ETH_MDIO: now also IC16.MDIO, R40.1; no longer IC17.MDIO, R43.1
- net FMC_A0: now also IC7.A0; no longer IC8.A0
- net FMC_A1: now also IC7.A1; no longer IC8.A1
- net FMC_A10: now also IC7.A10/AP; no longer IC8.A10/AP
- net FMC_A11: now also IC7.A11; no longer IC8.A11
- net FMC_A2: now also IC7.A2; no longer IC8.A2
- net FMC_A3: now also IC7.A3; no longer IC8.A3
- net FMC_A4: now also IC7.A4; no longer IC8.A4
- net FMC_A5: now also IC7.A5; no longer IC8.A5
- net FMC_A6: now also IC7.A6; no longer IC8.A6
- net FMC_A7: now also IC7.A7; no longer IC8.A7
- net FMC_A8: now also IC7.A8; no longer IC8.A8
- net FMC_A9: now also IC7.A9; no longer IC8.A9
- net FMC_BA0: now also IC7.BA0; no longer IC8.BA0
- net FMC_BA1: now also IC7.BA1; no longer IC8.BA1
- net FMC_D0: now also IC7.DQ0; no longer IC8.DQ0
- net FMC_D1: now also IC7.DQ1; no longer IC8.DQ1
- net FMC_D10: now also IC7.DQ10; no longer IC8.DQ10
- net FMC_D11: now also IC7.DQ11; no longer IC8.DQ11
- net FMC_D12: now also IC7.DQ12; no longer IC8.DQ12
- net FMC_D13: now also IC7.DQ13; no longer IC8.DQ13
- net FMC_D14: now also IC7.DQ14; no longer IC8.DQ14
- net FMC_D15: now also IC7.DQ15; no longer IC8.DQ15
- net FMC_D2: now also IC7.DQ2; no longer IC8.DQ2
- net FMC_D3: now also IC7.DQ3; no longer IC8.DQ3
- net FMC_D4: now also IC7.DQ4; no longer IC8.DQ4
- net FMC_D5: now also IC7.DQ5; no longer IC8.DQ5
- net FMC_D6: now also IC7.DQ6; no longer IC8.DQ6
- net FMC_D7: now also IC7.DQ7; no longer IC8.DQ7
- net FMC_D8: now also IC7.DQ8; no longer IC8.DQ8
- net FMC_D9: now also IC7.DQ9; no longer IC8.DQ9
- net FMC_NBL0: now also IC7.LDQM; no longer IC8.LDQM
- net FMC_NBL1: now also IC7.UDQM; no longer IC8.UDQM
- net FMC_SDCKE0: now also IC7.CKE; no longer IC8.CKE
- net FMC_SDCLK: now also IC7.CLK; no longer IC8.CLK
- net FMC_SDNCAS: now also IC7.!CAS; no longer IC8.!CAS
- net FMC_SDNE0: now also IC7.!CS, R24.2; no longer IC8.!CS, R25.2
- net FMC_SDNRAS: now also IC7.!RAS; no longer IC8.!RAS
- net FMC_SDNWE: now also IC7.!WE; no longer IC8.!WE
- net GND: now also C37.1, C38.2, C46.-, C47.2, C48.1, C50.2, C52.1, C56.2, C60.1, C61.2, C62.1, C63.2, C65.-, C66.2, IC12.TP, IC14.5WSX-, IC14.M1, IC14.M2, IC14.SX+, IC14.SY+, IC14.SY-, IC14.VSS, IC15.GND, IC16.AGND-15, IC16.AGND-19, IC16.DGND, IC16.IOGND-35, IC16.IOGND-47, IC7.GND-28, IC7.GND-54, IC7.GNDQ-12, IC7.GNDQ-46, IC7.GNDQ-52, IC7.GNDQ-6, IC8.A0, IC8.A1, IC8.A2, IC8.WP, R19.1, R27.2, R43.1, R56.1, SW1.2, SW2-1.C, SW2-2.1, X4-3.S; no longer C37.2, C38.1, C46.2, C47.-, C48.2, C50.1, C51.2, C56.1, C60.2, C61.1, C62.2, C63.1, C65.2, C66.-, C70.2, IC13.TP, IC14.GND, IC15.5WSX-, IC15.M1, IC15.M2, IC15.SX+, IC15.SY+, IC15.SY-, IC15.VSS, IC16.GND, IC17.AGND-15, IC17.AGND-19, IC17.DGND, IC17.IOGND-35, IC17.IOGND-47, IC8.GND-28, IC8.GND-54, IC8.GNDQ-12, IC8.GNDQ-46, IC8.GNDQ-52, IC8.GNDQ-6, IC9.A0, IC9.A1, IC9.A2, IC9.WP, R22.2, R23.2, R24.2, R30.2, R49.1, R59.1, SW1-1.C, SW1-2.1, SW2.2, X4-10.1, X4-12.1, X4-14.1, X4-16.1, X4-18.1, X4-20.1, X4-4.1, X4-6.1, X4-8.1
- net I2C1_SCL: now also IC14.SCK/SCL/TX, IC8.SCL; no longer IC15.SCK/SCL/TX, IC9.SCL
- net I2C1_SDA: now also IC14.SDI/SDA/RX, IC8.SDA; no longer IC15.SDI/SDA/RX, IC9.SDA
- net IRQ_TOUCH: now also IC14.SDO; no longer IC15.SDO
- net LCD_DISP: now also R32.1; no longer R35.1
- net LED_ACT: now also IC16.AN_EN(LED_ACT/COL), R44.2, R52.2; no longer IC17.AN_EN(LED_ACT/COL), R47.2, R55.2
- net LED_LINK: now also IC16.AN_0(LED_LINK), R51.2, R53.2; no longer IC17.AN_0(LED_LINK), R54.2, R56.2
- net LED_SPEED: now also IC16.AN_1(LED_SPEED), R49.2; no longer IC17.AN_1(LED_SPEED), R52.2
- net N$1: now also IC16.TX_CLK; no longer IC17.TX_CLK
- net N$10: now also IC16.TX_EN; no longer IC17.TX_EN
- net N$101: now also R47.2; no longer R50.2
- net N$102: now also C61.1, R45.1, R50.2; no longer C62.1, R48.1, R53.2
- net N$11: now also IC16.MII_MODE(RX_DV); no longer IC17.MII_MODE(RX_DV)
- net N$12: now also IC16.RX_CLK; no longer IC17.RX_CLK
- net N$13: now also R39.1; no longer R42.1
- net N$14: now also IC14.SIQ, R39.2; no longer IC15.SIQ, R42.2
- net N$15: now also IC16.TXD_0; no longer IC17.TXD_0
- net N$16: now also R26.1; no longer R29.1
- net N$166: now also IC12.VO-, R33.1; no longer IC13.VO-, R36.1
- net N$17: now also IC16.TXD_1; no longer IC17.TXD_1
- net N$171: now also IC12.IN-, R35.1, R38.2; no longer IC13.IN-, R38.1, R41.2
- net N$181: now also IC12.IN+, R33.2, R34.1; no longer IC13.IN+, R36.2, R37.1
- net N$19: now also R29.2; no longer R32.2
- net N$193: now also C50.1, R34.2; no longer C51.1, R37.2
- net N$194: now also C55.2, IC12.BYPASS; no longer C56.2, IC13.BYPASS
- net N$195: now also C51.1, R35.2; no longer C52.1, R38.2
- net N$2: now also R26.2; no longer R29.2
- net N$21: now also IC16.TXD_2; no longer IC17.TXD_2
- net N$22: now also IC16.X1; no longer IC17.X1
- net N$23: now also R48.2; no longer R51.2
- net N$25: now also R46.2; no longer R49.2
- net N$26: now also R43.2; no longer R46.2
- net N$27: now also IC16.PWR_DOWN/INT; no longer IC17.PWR_DOWN/INT
- net N$28: now also R57.2; no longer R60.2
- net N$29: now also IC16.TXD_3/SNI_MODE; no longer IC17.TXD_3/SNI_MODE
- net N$3: now also C59.1, R41.1, R42.2; no longer C60.1, R44.1, R45.2
- net N$30: now also IC10.VIN, R25.2; no longer IC11.VIN, R28.2
- net N$31: now also IC16.PHYAD4(RXD1_3); no longer IC17.PHYAD4(RXD1_3)
- net N$32: now also IC16.PHYAD3(RXD1_2); no longer IC17.PHYAD3(RXD1_2)
- net N$33: now also IC16.PHYAD0(COL); no longer IC17.PHYAD0(COL)
- net N$34: now also IC16.PHYAD2(RXD1_1); no longer IC17.PHYAD2(RXD1_1)
- net N$35: now also IC16.PHYAD1(RXD1_0); no longer IC17.PHYAD1(RXD1_0)
- net N$36: now also IC16.MDIX_EN(RX_ER); no longer IC17.MDIX_EN(RX_ER)
- net N$37: now also IC16.CRS/CRS_DV/LED_CFG; no longer IC17.CRS/CRS_DV/LED_CFG
- net N$4: now also C56.1, IC13.IO3, IC14.X-, R36.2; no longer C57.1, IC14.IO3, IC15.X-, R39.2
- net N$5: now also IC13.IO1, IC14.X+; no longer IC14.IO1, IC15.X+
- net N$50: now also IC12.VO+, R38.1; no longer IC13.VO+, R41.1
- net N$6: now also IC14.WAKE, R36.1; no longer IC15.WAKE, R39.1
- net N$7: now also C57.1, IC13.IO2, IC14.Y-; no longer C58.1, IC14.IO2, IC15.Y-
- net N$70: now also IC13.IO4, IC14.Y+; no longer IC14.IO4, IC15.Y+
- net N$8: now also R52.1; no longer R55.1
- net N$9: now also R53.1; no longer R56.1
- net N$97: now also IC16.RBIAS, R56.2; no longer IC17.RBIAS, R59.2
- net N$98: now also IC16.RESERVED-21, R54.2; no longer IC17.RESERVED-21, R57.2
- net N$99: now also IC16.RESERVED-20, R55.2; no longer IC17.RESERVED-20, R58.2
- net PFBOUT: now also C63.1, C65.+, C66.1, IC16.PFBIN1, IC16.PFBIN2, IC16.PFBOUT; no longer C65.1, C66.+, C67.1, IC17.PFBIN1, IC17.PFBIN2, IC17.PFBOUT
- net RD+: now also IC15.IO3, IC16.RD+, R45.2; no longer IC16.IO3, IC17.RD+, R48.2
- net RD-: now also IC15.IO4, IC16.RD-, R50.1; no longer IC16.IO4, IC17.RD-, R53.1
- net SDMMC1_CMD: now also R23.2; no longer R27.2
- net SDMMC1_D0: now also R22.2; no longer R26.2
- net SPI5_IRQ: now also IC4A.PA15; no longer IC4A.PB10, JP8.2
- net SW_WLED: now also IC10.SW; no longer IC11.SW
- net SYS_JTDO-SWO: now also IC6.IO4, X4-6.S; no longer IC7.IO4, X4-13.1
- net TCK: now also IC6.IO1, X4-2.S; no longer IC7.IO1, X4-9.1
- net TD+: now also IC15.IO1, IC16.TD+, R41.2; no longer IC16.IO1, IC17.TD+, R44.2
- net TD-: now also IC15.IO2, IC16.TD-, R42.1; no longer IC16.IO2, IC17.TD-, R45.1
- net TFT_BRIGHTNESS: now also IC10.CTRL; no longer IC11.CTRL
- net TMS: now also IC6.IO2, X4-4.S; no longer IC6.IO3, X4-7.1
- net USB_D_N: now also IC11.IO1, R30.1; no longer IC12.IO1, R33.1
- net USB_D_P: now also IC11.IO2, R31.1; no longer IC12.IO2, R34.1
- net USB_OTG_FS_D_N: now also R30.2; no longer R33.2
- net USB_OTG_FS_D_P: now also R31.2; no longer R34.2
- net USB_OTG_FS_ID: now also IC11.IO3; no longer IC12.IO3
- net USB_OTG_FS_PSO: now also IC9.EN; no longer IC10.EN
- net USB_OTG_FS_VBUS: now also C46.+, C48.2, IC11.VCC, IC9.OUT, R29.1; no longer C47.+, C49.2, IC10.OUT, IC12.VCC, R32.1
- net USER_SW: now also SW1.1; no longer SW2.1
- net VLED+: now also C45.1; no longer C46.1
- net VLED-: now also IC10.FB, R27.1; no longer IC11.FB, R30.1
Other:
- note added: "JTAG (SWD)"
- note added: "SDRAM"
- moved on the sheet: C35, C36, C37, C38, C39, C40, C41, C42, C43, C45, C48, C49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
