File: mcu/Eagle files/EEZ DIB MCU r2B1.brd (EAGLE design)
At the start: 139.5 x 70 mm, 181 parts, among them IC1 TPD4E001DRLR, IC10 TPD4E001DRLR, IC11 TPD4E001DRLR, IC12 TSC2007IPW, IC13 TPD4E001DRLR, IC14 DP83848CVV/NOPB, IC2 CD74HC4050PWR, IC3 STM32F769IGT6, IC4 LD1117ADT33TR, IC5 TPD4E001DRLR, IC6 IS42S16400J, IC7 AT24C256C-SSHL-B, IC8 TPS2051BDBVR, IC9 TPS61169DCKR, J1 503398-1892, J2 67803-8020, Q1 N.C., Q2 2N7002, SW1 TL1100CF160Q, SW2 PEC16-2215F-S0024, X1 DS1024-2*20R0, X2 DS1013-16SSIB1, X3 691322110005, X4 N.C., X5 LMJTAB881243M-L, Y1 25MHz, Y2 XTAL016178-85SMX

Commit message: MCU r2B1 with Ethernet and USB rotated
Parts:
- removed BOOT1: (no value), EEZ_Lib1:2MM-2
- added BOOT0: (no value), EEZ_Lib1:2MM-2
- IC13, IC5: value TPD4E001DRLR -> N.C.
- moved EEZ_SIGNATURE 97.7 mm to (-0.82, 23.0)
- moved J2 69.3 mm to (96.7, 67.2), turned to 270 degrees
- moved C38 65.0 mm to (76.6, 5.66), turned to 180 degrees
- moved IC5 62.8 mm to (79.9, 5.77), turned to 180 degrees
- moved VBUS 61.6 mm to (106.4, 64.6), turned to 0 degrees
- moved C51 61.4 mm to (104.2, 64.6), turned to 270 degrees
- moved R24 60.4 mm to (108.5, 64.6), turned to 90 degrees
- moved Q1 57.5 mm to (108.3, 60.3), turned to 0 degrees
- moved JP5 56.2 mm to (91.2, 8.17), turned to 90 degrees
- moved X4 53.4 mm to (81.8, 10.1), turned to 180 degrees
- moved IC10 50.9 mm to (96.2, 57.7), turned to 180 degrees
- moved R18 50.0 mm to (91.4, 11.3), turned to 270 degrees
- moved R27 49.8 mm to (102.7, 57.3), turned to 0 degrees
- moved IC8 48.8 mm to (87.4, 60.8)
- moved C49 48.7 mm to (86.8, 63.7)
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Connections:
- net +3V3: now also BOOT0.2; no longer BOOT1.2
- net BOOT0: now also BOOT0.1; no longer BOOT1.1
Routing:
- net USB_OTG_FS_PSO: track 53.3 -> 12.7 mm, vias 2 -> 0
- net +5V: track 161.0 -> 121.4 mm
- net !USB_OTG_FS_OC: track 53.4 -> 16.5 mm
- net TCK: track 18.6 -> 54.9 mm, vias 0 -> 2
- net SYS_JTDO-SWO: track 37.6 -> 63.1 mm
- net PE: track 168.1 -> 148.6 mm
- net !RESET: track 229.9 -> 245.6 mm, vias 12 -> 13
- net TMS: track 29.8 -> 41.9 mm
- net USB_D_P: track 33.9 -> 27.4 mm
- net I2C1_SDA: track 130.3 -> 123.9 mm, vias 8 -> 7
- net USB_D_N: track 34.1 -> 28.6 mm
- net ENC_B: track 43.1 -> 38.1 mm, vias 2 -> 0
- net DAC_OUT1: track 43.7 -> 48.0 mm
- net I2C1_SCL: track 127.2 -> 122.9 mm, vias 6 -> 5
- net ENC_SW: track 83.9 -> 79.7 mm
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