File: mcu/Eagle files/EEZ DIB MCU r2B3.brd (EAGLE design)
At the start: 139.5 x 70 mm, 181 parts, among them IC1 TPD4E001DRLR, IC10 TPD4E001DRLR, IC11 TPD4E001DRLR, IC12 TSC2007IPW, IC13 TPD4E001DRLR, IC14 DP83848CVV/NOPB, IC2 CD74HC4050PWR, IC3 STM32F769IGT6, IC4 LD1117ADT33TR, IC5 TPD4E001DRLR, IC6 IS42S16400J, IC7 AT24C256C-SSHL-B, IC8 TPS2051BDBVR, IC9 TPS61169DCKR, J1 503398-1892, J2 67803-8020, Q1 N.C., Q2 2N7002, SW1 TL1100CF160Q, SW2 PEC16-2215F-S0024, X1 DS1024-2*20R0, X2 DS1013-16SSIB1, X3 691322110005, X4 N.C., X5 LMJTAB881243M-L, Y1 25MHz, Y2 XTAL016178-85SMX

Commit message: #62
Parts:
- added SW3: EVQP7A01P, EEZ_switches:PANASONIC_EVQP
- added U$3: HR000002, OSHWA:CERT-SMALL-SILK
- IC11, IC13, IC5: value TPD4E001DRLR -> N.C.
- moved BOOT1 107.7 mm to (1.23, 29.6), turned to 270 degrees
- moved C13 52.8 mm to (3.95, 16.6), turned to 90 degrees
- moved C15 52.7 mm to (16.6, 14.0), turned to 90 degrees
- moved IC4 50.6 mm to (11.8, 8.29), turned to 180 degrees
- moved X5 50.4 mm to (15.9, 59.5), turned to 180 degrees
- moved C14 47.9 mm to (9.86, 15.9)
- moved R44 47.5 mm to (26.6, 63.3)
- moved R43 47.4 mm to (28.5, 63.3)
- moved R38 47.4 mm to (32.5, 63.3), turned to 90 degrees
- moved SPEED 44.8 mm to (30.5, 63.3)
- moved C61 29.6 mm to (20.5, 47.3), turned to 180 degrees
- moved C59 26.9 mm to (12.0, 47.5), turned to 0 degrees
- moved IC13 25.8 mm to (15.9, 46.9), turned to 180 degrees
- moved C57 22.9 mm to (13.1, 45.5), turned to 180 degrees
- moved D1 21.7 mm to (0.90, 32.7), turned to 0 degrees
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Connections:
- net +3V3: now also SW3.2.1, SW3.2.2
- net BOOT0: now also SW3.1.1, SW3.1.2; no longer X2.2
Routing:
- net +5V: track 246.6 -> 161.0 mm, vias 13 -> 12
- net BOOT0: track 115.2 -> 176.7 mm
- net LED_SPEED: track 14.9 -> 68.5 mm
- net LED_ACT: track 18.3 -> 67.1 mm
- net LED_LINK: track 18.7 -> 64.0 mm
- net !FAULT: track 231.8 -> 273.4 mm, vias 7 -> 10
- net RD+: track 37.5 -> 21.2 mm, vias 3 -> 2
- net RD-: track 36.2 -> 21.0 mm, vias 3 -> 2
- net N$9: track 20.6 -> 7.11 mm
- net PWR_DIRECT: track 108.0 -> 121.3 mm
- net PWR_SSTART: track 110.0 -> 119.3 mm
- net TD-: track 33.1 -> 24.3 mm
- net !RESET: track 238.4 -> 229.9 mm, vias 13 -> 12
- net TD+: track 35.2 -> 28.7 mm
- net +VAUX: track 188.3 -> 194.3 mm
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- added copper zone on layer 1, net +5V
Other:
- board text added: "EEZ DIB MCU (01/2020 r2B3)"
- board text added: "EEZ DIB MCU (01/2020 r2B3) Project source code: github.com/eez-open/modular-psu"
- board text removed: "EEZ DIB MCU (12/2019 r1B6)"
- board text removed: "Project source code: github.com/eez-open/modular-psu"
