File: mcu/Eagle files/EEZ DIB MCU r2B3.sch (EAGLE design)
At the start: 177 parts, among them IC1 TPD4E001DRLR, IC10 TPD4E001DRLR, IC11 TPD4E001DRLR, IC12 TSC2007IPW, IC13 TPD4E001DRLR, IC14 DP83848CVV/NOPB, IC2 CD74HC4050PWR, IC3 STM32F769IGT6, IC4 LD1117ADT33TR, IC5 TPD4E001DRLR, IC6 IS42S16400J, IC7 AT24C256C-SSHL-B, IC8 TPS2051BDBVR, IC9 TPS61169DCKR, J1 503398-1892, J2 67803-8020, Q1 N.C., Q2 2N7002, SW1 TL1100CF160Q, SW2 PEC16-2215F-S0024, X1 DS1024-2*20R0, X2 DS1013-16SSIB1, X3 691322110005, X4 N.C., X5 LMJTAB881243M-L, Y1 25MHz, Y2 XTAL016178-85SMX

Commit message: #62
Parts:
- added SW3: EVQP7A01P, EEZ_switches:EVQP7A01P
- added U$3: HR000002, OSHWA:CERT-SMALL
- IC11, IC13, IC5: value TPD4E001DRLR -> N.C.
Connections:
- net +3V3: now also SW3.2
- net BOOT0: now also SW3.1; no longer X2-2.1
Other:
- note added: "2 N.C."
- note added: "MCU BOOT0 switch"
- note removed: "2 MBOOT"
Changed lines of the file:
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@@
 <part name="+3V9" library="supply1" deviceset="+3V3" device=""/>
 <part name="JP12" library="EEZ_Lib1" deviceset="JP2-NOCUT" device=""/>
-<part name="IC13" library="EEZ_Lib1" deviceset="TPD4E001" device="-DRL" value="TPD4E001DRLR"/>
+<part name="IC13" library="EEZ_Lib1" deviceset="TPD4E001" device="-DRL" value="N.C."/>
 <part name="+3V10" library="supply1" deviceset="+3V3" device=""/>
 <part name="C57" library="rcl" deviceset="C-EU" device="C0603" value="N.C."/>
@@
 <part name="SUPPLY18" library="supply2" deviceset="GND" device=""/>
 <part name="SUPPLY17" library="supply2" deviceset="GND" device=""/>
-<part name="IC5" library="EEZ_Lib1" deviceset="TPD4E001" device="-DRL" value="TPD4E001DRLR"/>
+<part name="IC5" library="EEZ_Lib1" deviceset="TPD4E001" device="-DRL" value="N.C."/>
 <part name="SUPPLY25" library="supply2" deviceset="GND" device=""/>
 <part name="+3V310" library="supply1" deviceset="+3V3" device=""/>
@@
 <part name="R23" library="rcl" deviceset="R-EU_" device="R0805" value="10R"/>
 <part name="C50" library="rcl" deviceset="C-EU" device="C0805" value="2u2"/>
-<part name="IC11" library="EEZ_Lib1" deviceset="TPD4E001" device="-DRL" value="TPD4E001DRLR"/>
+<part name="IC11" library="EEZ_Lib1" deviceset="TPD4E001" device="-DRL" value="N.C."/>
 <part name="+3V314" library="supply1" deviceset="+3V3" device=""/>
 <part name="C54" library="rcl" deviceset="C-EU" device="C0603" value="N.C."/>
@@
 <part name="P+2" library="supply1" deviceset="+5V" device=""/>
 <part name="C8" library="rcl" deviceset="C-EU" device="C0805" value="1n"/>
+<part name="+3V7" library="supply1" deviceset="+3V3" device=""/>
+<part name="SW3" library="EEZ_switches" deviceset="EVQP7A01P" device=""/>
+<part name="U$3" library="OSHWA" deviceset="CERT" device="-SMALL" value="HR000002"/>
 </parts>
 <sheets>
@@
 <circle x="110.49" y="151.13" radius="0.635" width="0.1524" layer="101"/>
 <circle x="110.49" y="148.59" radius="0.635" width="0.1524" layer="101"/>
-<text x="113.03" y="158.115" size="1.4224" layer="101">2 MBOOT</text>
+<text x="113.03" y="158.115" size="1.4224" layer="101">2 N.C.</text>
 <text x="105.41" y="151.765" size="1.4224" layer="101" rot="R180">Gnd 7</text>
 <text x="113.03" y="153.035" size="1.4224" layer="101">6 +5V</text>
@@
 <attribute name="VALUE" x="105.41" y="97.79" size="1.778" layer="96" rot="MR180"/>
 </instance>
+<instance part="U$3" gate="G$1" x="8.255" y="10.795" smashed="yes">
+<attribute name="VALUE" x="2.286" y="8.255" size="1.778" layer="94" font="vector" ratio="12"/>
+</instance>
 </instances>
 <busses>
@@
 </segment>
 </net>
-<net name="BOOT0" class="0">
-<segment>
-<pinref part="X2" gate="-2" pin="1"/>
-<wire x1="60.96" y1="154.94" x2="78.74" y2="154.94" width="0.1524" layer="91"/>
-<label x="78.74" y="155.575" size="1.27" layer="102" rot="MR0"/>
-</segment>
-</net>
 <net name="N$7" class="0">
 <segment>
@@
 <text x="6.35" y="75.565" size="1.778" layer="97">Resistive touchscreen controller</text>
 <wire x1="157.48" y1="78.74" x2="157.48" y2="35.56" width="0.1524" layer="97" style="shortdash"/>
-<wire x1="264.16" y1="96.52" x2="157.48" y2="96.52" width="0.1524" layer="97" style="shortdash"/>
+<wire x1="264.16" y1="96.52" x2="215.9" y2="96.52" width="0.1524" layer="97" style="shortdash"/>
 <text x="160.02" y="91.44" size="1.778" layer="97">Audio output</text>
+<wire x1="215.9" y1="96.52" x2="157.48" y2="96.52" width="0.1524" layer="97" style="shortdash"/>
 <wire x1="96.52" y1="177.8" x2="96.52" y2="78.74" width="0.1524" layer="97" style="shortdash"/>
 <rectangle x1="184.15" y1="142.875" x2="191.77" y2="146.685" layer="97" rot="R180"/>
@@
 <text x="84.455" y="170.815" size="1.27" layer="100">+28.6V</text>
 <rectangle x1="229.235" y1="113.665" x2="235.585" y2="120.65" layer="97"/>
+<text x="218.44" y="91.44" size="1.778" layer="97">MCU BOOT0 switch</text>
+<wire x1="215.9" y1="96.52" x2="215.9" y2="38.1" width="0.1524" layer="97" style="shortdash"/>
 </plain>
 <instances>
@@
 <attribute name="VALUE" x="182.88" y="46.99" size="1.778" layer="96"/>
 </instance>
+<instance part="+3V7" gate="G$1" x="256.54" y="58.42" smashed="yes" rot="R270">
+<attribute name="VALUE" x="253.365" y="54.61" size="1.778" layer="96"/>
+</instance>
+<instance part="SW3" gate="G$1" x="241.3" y="58.42" smashed="yes">
+<attribute name="NAME" x="238.76" y="62.23" size="1.778" layer="95"/>
+<attribute name="VALUE" x="235.585" y="55.245" size="1.778" layer="96"/>
+</instance>
 </instances>
 <busses>
@@
 <wire x1="134.62" y1="165.1" x2="134.62" y2="162.56" width="0.1524" layer="91"/>
 </segment>
+<segment>
+<pinref part="+3V7" gate="G$1" pin="+3V3"/>
+<pinref part="SW3" gate="G$1" pin="2"/>
+<wire x1="246.38" y1="58.42" x2="254" y2="58.42" width="0.1524" layer="91"/>
+</segment>
 </net>
 <net name="GND" class="2">
@@
 </segment>
 </net>
+<net name="BOOT0" class="0">
+<segment>
+<label x="220.98" y="59.055" size="1.27" layer="102"/>
+<pinref part="SW3" gate="G$1" pin="1"/>
+<wire x1="236.22" y1="58.42" x2="220.98" y2="58.42" width="0.1524" layer="91"/>
+</segment>
+</net>
