File: bp3c/Eagle files/EEZ DIB BP3C r1B5.brd (EAGLE design)
At the start: 110 x 85 mm, 30 parts, among them Q1 IRLML6244TRPBF, Q2 IRLML6244TRPBF, X1 ZL202-20G, X2 ZL202-20G, X3 ZL202-20G, X4 ZL212-40KG, X5 TSW-113-07-F-D, X6 TSW-113-07-F-D, X7 TSW-113-07-F-D

Commit message: #34
Parts:
- added JP1, JP5, JP8, JP9: JP2-CUT, EEZ_Lib1:JP2-CUT
- added JP2, JP3, JP4, JP6, JP7: JP2-NOCUT, EEZ_Lib1:JP2-NOCUT
Connections:
- new net N$11: JP4.1, X6.18
- new net N$13: JP8.2, X6.19
- new net N$14: JP6.1, X7.18
- new net N$15: JP5.2, X7.17
- new net N$16: JP9.2, X7.19
- new net N$2: JP1.2, X5.17
- new net N$5: JP7.2, X5.19
- new net N$6: JP2.1, X5.18
- new net N$9: JP3.2, X6.17
- net GND: now also JP1.1, JP2.2, JP3.1, JP4.2, JP5.1, JP6.2, JP7.1, JP8.1, JP9.1; no longer X5.18, X5.19, X6.19, X7.17, X7.19
Routing:
- net N$14: track 0.00 -> 6.38 mm
- net N$6: track 0.00 -> 6.31 mm
- net N$11: track 0.00 -> 6.25 mm
- net N$16: track 0.00 -> 2.64 mm
- net N$5: track 0.00 -> 2.64 mm
- net N$15: track 0.00 -> 2.59 mm
- net N$2: track 0.00 -> 2.59 mm
- net N$13: track 0.00 -> 2.58 mm
- net N$9: track 0.00 -> 2.53 mm
Other:
- board text added: "EEZ DIB BP3C (05/2019 r1B5)"
- board text removed: "EEZ DIB BP3C (02/2019 r1B5)"
