File: bp3c/Eagle files/EEZ DIB BP3C r2B1.brd (EAGLE design)
At the start: 110 x 85 mm, 39 parts, among them Q1 IRLML6244TRPBF, Q2 IRLML6244TRPBF, X1 ZL202-20G, X2 ZL202-20G, X3 ZL202-20G, X4 ZL212-40KG, X5 TSW-113-07-F-D, X6 TSW-113-07-F-D, X7 TSW-113-07-F-D

Commit message: #36
Parts:
- removed D3: BAS316, EEZ_Lib1:SOD323-R
- added C1: 100n, rcl:C0603
- added IC1: PCA9536D, EEZ_DIB:SOIC127P600X173-8N
- D2: value N.C. -> BAS316
- moved D2 10.6 mm to (21.8, 16.0), turned to 0 degrees
Connections:
- net +3V3: now also C1.1, IC1.8
- net +5V: now also D2.C; no longer D3.C
- net GND: now also C1.2, IC1.4
- net I2C1_SCL: now also IC1.6
- net I2C1_SDA: now also IC1.7
- net N$101: no longer D2.C
- net N$104: now also D2.A; no longer D3.A
- net OUT_PAR: now also IC1.1; no longer D2.A, X4.4
- net OUT_SER: now also IC1.2; no longer X4.3
Routing:
- net I2C1_SDA: track 116.4 -> 148.4 mm, vias 1 -> 2
- net I2C1_SCL: track 114.0 -> 142.0 mm, vias 1 -> 2
- net OUT_SER: track 45.8 -> 20.4 mm
- net +3V3: track 113.6 -> 136.9 mm
- net OUT_PAR: track 49.5 -> 32.2 mm
- net GND: track 54.3 -> 39.9 mm, vias 77 -> 82
- net +5V: track 290.5 -> 291.4 mm
- net SPI5_CSA: track 112.0 -> 111.3 mm
Other:
- board text added: "EEZ DIB BP3C (05/2019 r2B1)"
- board text removed: "EEZ DIB BP3C (05/2019 r1B5)"
