File: dcm220/Eagle files/EEZ DIB DCM220 r2B6.brd (EAGLE design)
At the start: 155 x 95 mm, 245 parts, among them IC1 Si8662AB-B-IS1, IC10 MC33272ADR2G, IC11 LT3763EFE#PBF, IC12 MC33274ADR2G, IC13 LT3763EFE#PBF, IC2 TPS54060DGQ, IC3 Si8641AB-B-IS1, IC4 M24C32-WMN6P, IC5 LP2985-33DBVR, IC6 74HC2G04GW,125, IC7 N.C., IC8 STM32F373C8T6, IC9 TL431B, J1 4907, J2 571-0500, J3 571-0100, J4 571-0500, J5 571-0100, Q1 BSP716NH6327XTSA1, Q10 BSS84, Q2 NTD5867NLT4G, Q3 NTD5867NLT4G, Q4 BSS205NH6327XTSA1, Q5 BSS84, Q6 BSP716NH6327XTSA1, Q7 NTD5867NLT4G, Q8 NTD5867NLT4G, Q9 BSS205NH6327XTSA1, X1 39-30-1020, X2 77317-104-28LF, X3 N.C., X4 DS1024-2*5R0, Y1 LF XTAL026392

Commit message: #53 (DCM220 r2B6)
Parts:
- added TX_PU: 10K, rcl:R0805
- moved R23 4.17 mm to (119.3, 33.8)
- moved C39 2.79 mm to (116.3, 34.9), turned to 0 degrees
- moved IC9 2.30 mm to (116.3, 32.1)
Connections:
- net +3V3: now also TX_PU.2
- net DIB_UART_RX: now also X2.27; no longer X2.28
- net DIB_UART_TX: now also X2.28; no longer X2.27
- net MISO: now also IC8.26; no longer IC8.30
- net MOSI: now also IC8.27; no longer IC8.31
- net SCLK: now also IC8.28; no longer IC8.29
- net UART_RX: now also IC8.31; no longer IC8.13
- net UART_TX: now also IC8.30, TX_PU.1; no longer IC8.12
Routing:
- net +3V3: track 433.0 -> 440.7 mm
- net MISO: track 54.5 -> 49.6 mm, vias 4 -> 2
- net SCLK: track 40.6 -> 36.3 mm
- net UART_TX: track 44.5 -> 42.3 mm
- net DIB_UART_TX: track 9.92 -> 8.06 mm
- net +VREF: track 20.5 -> 19.4 mm
- net DIB_UART_RX: track 9.51 -> 10.6 mm, vias 1 -> 0
- net TEMP#2: track 47.0 -> 46.1 mm
Other:
- board text added: "EEZ DIB DCM220 (11/2019 r2B6)"
- board text added: "EEZ DIB DCM220 (11/2019 r2B6) Project source code: github.com/eez-open"
- board text removed: "EEZ DIB DCM220 (10/2019 r2B5)"
- board text removed: "EEZ DIB DCM220 (10/2019 r2B5) Project source code: github.com/eez-open"

Commit message: DCM220 BOM update
Other:
- board text added: "EEZ DIB DCM220 (12/2019 r2B6)"
- board text added: "EEZ DIB DCM220 (12/2019 r2B6) Project source code: github.com/eez-open"
- board text removed: "EEZ DIB DCM220 (11/2019 r2B6)"
- board text removed: "EEZ DIB DCM220 (11/2019 r2B6) Project source code: github.com/eez-open"
Changed lines of the file:
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@@
 <rectangle x1="131.9967" y1="86.1921" x2="132.2367" y2="86.1959" layer="21"/>
 <text x="135.5625" y="82.3555" size="1.27" layer="21" font="vector" ratio="10" rot="SR0">EEZ DIB DCM220
-(11/2019 r2B6)</text>
-<text x="151.164" y="88.134" size="1.27" layer="22" font="vector" ratio="10" rot="SMR0">EEZ DIB DCM220 (11/2019 r2B6)
+(12/2019 r2B6)</text>
+<text x="151.164" y="88.134" size="1.27" layer="22" font="vector" ratio="10" rot="SMR0">EEZ DIB DCM220 (12/2019 r2B6)
 Project source code: github.com/eez-open</text>
 <rectangle x1="129.54" y1="86.741" x2="151.638" y2="92.3925" layer="21"/>
