File: aux-ps/EDA files/EEZ DIB AUX PS r3B6.brd (EAGLE design)
At the start: 230.5 x 60 mm, 93 parts, among them IC1 BD00FC0WFP-E2, IC2 MAX31760AEE+, J1 PF0030/PC, J2 1-726388-2, J3 1-726388-2, J4 SWEB 8094 AU/GN, K1 RT424005, K2 RT424005, Q1 MMBT5551, Q2 MMBT5551, Q3 2N7002, SW1 DF62J12S2AHQA, X1 39-28-1063, X2 39-30-1039, X3 DS1013-16SSIB1, X4 47053-1000, X5 N.C.

Commit message: #103
Routing:
- net PE: track 501.8 -> 502.2 mm, vias 1 -> 2
Other:
- board text added: "EEZ DIB AUX PS (03/2021 r3B6)"
- board text added: "EEZ DIB AUX PS (03/2021 r3B6) Project source code: github.com/eez-open/modular-psu"
- board text removed: "EEZ DIB AUX PS (12/2020 r3B5)"
- board text removed: "EEZ DIB AUX PS (12/2020 r3B5) Project source code: github.com/eez-open/modular-psu"
Changed lines of the file:
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@@
 <setting verticaltext="up"/>
 </settings>
-<grid distance="0.5" unitdist="mil" unit="mil" style="lines" multiple="10" display="no" altdistance="12.5" altunitdist="mil" altunit="mil"/>
+<grid distance="2.5" unitdist="mil" unit="mil" style="lines" multiple="10" display="no" altdistance="12.5" altunitdist="mil" altunit="mil"/>
 <layers>
 <layer number="1" name="Top" color="11" fill="1" visible="yes" active="yes"/>
@@
 <layer number="131" name="tAdjust" color="7" fill="1" visible="no" active="no"/>
 <layer number="132" name="bAdjust" color="7" fill="1" visible="no" active="no"/>
-<layer number="133" name="DNP_top" color="12" fill="1" visible="yes" active="yes"/>
+<layer number="133" name="DNP_top" color="12" fill="1" visible="no" active="yes"/>
 <layer number="144" name="Drill_legend" color="7" fill="1" visible="no" active="no"/>
 <layer number="148" name="Document_mirrored" color="7" fill="1" visible="no" active="no"/>
@@
 <rectangle x1="16.5537" y1="30.0906" x2="16.7937" y2="30.0944" layer="21"/>
 <text x="29.464" y="2.667" size="1.1684" layer="21" font="vector" ratio="10" rot="SR0">EEZ DIB AUX PS
-(12/2020 r3B5)
+(03/2021 r3B6)
 Project source code: github.com/eez-open/modular-psu</text>
 <wire x1="1.5" y1="0" x2="229" y2="0" width="0.1" layer="20"/>
@@
 <vertex x="175.5525" y="54.739"/>
 </polygon>
-<text x="227.195" y="46.609" size="1.27" layer="16" ratio="10" rot="MR270">EEZ DIB AUX PS (12/2020 r3B5)</text>
+<text x="227.195" y="46.609" size="1.27" layer="16" ratio="10" rot="MR270">EEZ DIB AUX PS (03/2021 r3B6)</text>
 <wire x1="12.0015" y1="22.0345" x2="0.1905" y2="22.0345" width="0.254" layer="21"/>
 <wire x1="12.0015" y1="20.5105" x2="0.1905" y2="20.5105" width="0.254" layer="21" style="shortdash"/>
@@
 <dimension x1="0.5" y1="0" x2="4.5" y2="60" x3="-2.359" y3="30" textsize="2" layer="47" dtype="vertical"/>
 <wire x1="12.0015" y1="10.9855" x2="0.1905" y2="10.9855" width="0.254" layer="21"/>
-<dimension x1="-6" y1="0" x2="10" y2="45.5" x3="-21.359" y3="22.75" textsize="2" layer="47" dtype="vertical"/>
-<dimension x1="-6" y1="0" x2="15.5" y2="27" x3="-16.859" y3="13.5" textsize="2" layer="47" dtype="vertical"/>
-<dimension x1="-12.5" y1="0" x2="20" y2="16" x3="-12.359" y3="8" textsize="2" layer="47" dtype="vertical"/>
+<dimension x1="-6" y1="0" x2="5.5" y2="45.5" x3="-21.359" y3="22.75" textsize="2" layer="47" dtype="vertical"/>
+<dimension x1="-6" y1="0" x2="6.5" y2="27" x3="-16.859" y3="13.5" textsize="2" layer="47" dtype="vertical"/>
+<dimension x1="-12.5" y1="0" x2="27.5" y2="16.5" x3="-12.359" y3="8.25" textsize="2" layer="47" dtype="vertical"/>
 <dimension x1="-10.5" y1="0" x2="5.5" y2="6" x3="-7.859" y3="3" textsize="2" layer="47" dtype="vertical"/>
 <dimension x1="-1.5" y1="-3.5" x2="0" y2="0" x3="-0.75" y3="-2.5" textsize="2" layer="47" dtype="horizontal"/>
@@
 <wire x1="173.9265" y1="7.4295" x2="174.1805" y2="7.6835" width="0.6096" layer="16"/>
 <wire x1="174.1805" y1="7.6835" x2="174.625" y2="8.9535" width="0.6096" layer="16"/>
-<wire x1="183.722" y1="42.552" x2="186.7535" y2="42.672" width="1.6764" layer="16"/>
-<wire x1="186.7535" y1="42.672" x2="187.3885" y2="43.307" width="1.6764" layer="16"/>
+<wire x1="186.6335" y1="42.552" x2="187.3885" y2="43.307" width="1.6764" layer="16"/>
 <wire x1="187.3885" y1="43.307" x2="197.8025" y2="43.307" width="1.6764" layer="16"/>
 <wire x1="199" y1="37" x2="199" y2="42.1095" width="1.6764" layer="16"/>
@@
 <wire x1="200.127" y1="4.318" x2="196.7865" y2="4.318" width="0.6096" layer="1"/>
 <wire x1="196.7865" y1="4.318" x2="195.326" y2="2.8575" width="0.6096" layer="1"/>
+<wire x1="183.722" y1="42.552" x2="186.6335" y2="42.552" width="1.6764" layer="16"/>
 </signal>
 <signal name="+5V">
@@
 <wire x1="193.749" y1="44.1325" x2="200.533" y2="44.1325" width="2.032" layer="1"/>
 <wire x1="200.533" y1="44.1325" x2="211" y2="44.1325" width="2.032" layer="1"/>
-<wire x1="211" y1="44.1325" x2="211" y2="30" width="2.032" layer="1"/>
-<wire x1="211" y1="44.1325" x2="211" y2="56.0175" width="2.032" layer="1"/>
-<wire x1="211" y1="56.0175" x2="209.9945" y2="57.023" width="2.032" layer="1"/>
+<wire x1="211" y1="44.1325" x2="211" y2="30" width="2.54" layer="1"/>
 <wire x1="219.9005" y1="57.023" x2="215.0745" y2="57.023" width="2.032" layer="16"/>
 <wire x1="200.5965" y1="47.4255" x2="200.5965" y2="44.196" width="2.032" layer="1"/>
@@
 <wire x1="153.162" y1="16.764" x2="147.955" y2="16.764" width="0.6096" layer="1"/>
 <wire x1="147.955" y1="16.764" x2="147.8915" y2="16.8275" width="0.6096" layer="1"/>
+<via x="211.5" y="49.5" extent="1-16" drill="3.2" diameter="5.5"/>
+<wire x1="209.9945" y1="57.023" x2="209.9945" y2="51.0055" width="2.54" layer="1"/>
+<wire x1="209.9945" y1="51.0055" x2="211.5" y2="49.5" width="2.54" layer="1"/>
+<wire x1="211" y1="44.1325" x2="211" y2="49" width="2.54" layer="1"/>
+<wire x1="211" y1="49" x2="211.5" y2="49.5" width="2.032" layer="1"/>
 <wire x1="25.527" y1="16.51" x2="29.3" y2="21.58" width="0" layer="19" extent="1-1"/>
 <wire x1="25.5" y1="16.5" x2="25.527" y2="16.51" width="0" layer="19" extent="1-16"/>
@@
 <wire x1="15" y1="5.5" x2="19.14" y2="11.42" width="0" layer="19" extent="1-1"/>
 </signal>
-<signal name="HOLE_UR">
-<via x="211.5" y="5.5" extent="1-16" drill="3.2" diameter="5.5"/>
-</signal>
 <signal name="HOLE_UM">
 <via x="120" y="49.5" extent="1-16" drill="3.2" diameter="5.5"/>
@@
 <wire x1="67.879" y1="38.608" x2="68.0695" y2="38.7985" width="0.254" layer="1"/>
 </signal>
+<signal name="N$22">
+<via x="211.5" y="5.5" extent="1-16" drill="3.2" diameter="5.5"/>
+</signal>
 </signals>
